File: ver1/hardware/4bit-addr/TB04addr4bitVer3.kicad_pcb (KiCad board)
At the start: 2 copper layers, 220 x 180 mm, 176 parts, among them IC1 74HC161N, IC2 74HC161N, IC3 74HC161N, IC4 74HC161N, IC5 74HC161N, IC6 74HC161N, IC7 74HC161N, IC8 74HC161N, IC9 74HC161N, J1 USB_C_Receptacle_PowerOnly_6P, J2 Conn_01x06_Socket, J3 Conn_02x05_Odd_Even, SW1 SW_SPDT, SW2 SW_DIP_x04, SW3 SW_DIP_x04, SW4 SW_DIP_x04, SW5 SW_SPDT, SW6 SW_Push, SW7 SW_Push, U1 74LS253, U10 OSC8MI/H, U11 74LS273, U12 4040, U13 4040, U14 74HC238, U15 74HC138, U16 74HC00, U17 74HC14, U18 74LS273, U19 74LS273, U2 74LS253, U20 74HC273, U21 74HC74, U22 28C256, U23 28C256, U24 28C256, U3 74LS253, U4 74LS253, U5 28C256, U6 74LS253, U7 74LS253, U8 74LS253, U9 74LS253

Commit message: 4bitCPUの回路図を修正（PCBは工事中）
Co-Authored-By: Claude Opus 4.8 <noreply@anthropic.com>
Connections:
- RN8 pad 2: Net-(D38-K) -> Net-(D39-K)
- RN8 pad 3: Net-(D39-K) -> Net-(D40-K)
- RN8 pad 4: Net-(D40-K) -> Net-(D41-K)
- RN8 pad 5: Net-(D41-K) -> Net-(D38-K)
- U1 pad 2: Reg_RD_SEL0b -> Reg_RD_SEL1a
- U14 pad 12: WB -> Execute
- U14 pad 13: Execute -> Decord
- U14 pad 14: Decord -> Fetch
- U14 pad 15: Fetch -> WB
- U15 pad 6: WB -> Execute
- U16 pad 9: WB -> Decord
- U2 pad 2: Reg_RD_SEL0b -> Reg_RD_SEL1a
- U3 pad 14: Reg_RD_SEL1a -> Reg_RD_SEL0b
- U4 pad 14: Reg_RD_SEL1a -> Reg_RD_SEL0b
Routing:
- net WB: track 141.9 -> 5.67 mm, vias 4 -> 1
- net Execute: track 245.1 -> 345.9 mm, vias 4 -> 6
- net Fetch: track 112.6 -> 100.3 mm, vias 2 -> 1
- net Decord: track 96.8 -> 107.6 mm
