File: ver1/hardware/4bit-addr/ROM_ALU_Decoder.kicad_sch (KiCad schematic)
At the start: 31 parts, among them IC9 74HC161N, U11 74LS273, U14 74HC238, U18 74LS273, U19 74LS273, U20 74HC273, U21 74HC74, U22 28C256, U23 28C256, U24 28C256, U5 28C256

Commit message: 4bitCPUの回路図を修正（PCBは工事中）
Co-Authored-By: Claude Opus 4.8 <noreply@anthropic.com>
Connections:
- net Decord: now also U14.13 (Y2); no longer U14.14 (Y1)
- net Execute: now also U14.12 (Y3); no longer U14.13 (Y2)
- net Fetch: now also U14.14 (Y1); no longer U14.15 (Y0)
- net WB: now also U14.15 (Y0); no longer U14.12 (Y3)
- net at D41.1 (K): now also RN8.4 (R3); no longer RN8.5 (R4)
- net at D40.1 (K): now also RN8.3 (R2); no longer RN8.4 (R3)
- net at D38.1 (K): now also RN8.5 (R4); no longer RN8.2 (R1)
- net at D39.1 (K): now also RN8.2 (R1); no longer RN8.3 (R2)
Other:
- note added: "rev.1 １命令めでフェッチを確実にするために入れ替えた"
- moved on the sheet: D38, D39, D40, D41
Changed lines of the file:
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@@
 	(generator_version "9.0")
 	(paper "A3")
+	(text "rev.1    １命令めでフェッチを確実にするために入れ替えた"
+		(exclude_from_sim no)
+		(at 162.052 141.478 0)
+		(effects
+			(font
+				(size 1.27 1.27)
+			)
+		)
+	)
 	(text "フェーズ発生器"
 		(exclude_from_sim no)
@@
 	(global_label "Decord"
 		(shape output)
-		(at 153.67 147.32 0)
+		(at 153.67 149.86 0)
 		(fields_autoplaced yes)
 		(effects
@@
 		)
 		(property "Intersheetrefs" "${INTERSHEET_REFS}"
-			(at 163.1866 147.32 0)
+			(at 163.1866 149.86 0)
 			(effects
 				(font
@@
 	(global_label "Execute"
 		(shape output)
-		(at 153.67 149.86 0)
+		(at 153.67 152.4 0)
 		(fields_autoplaced yes)
 		(effects
@@
 		)
 		(property "Intersheetrefs" "${INTERSHEET_REFS}"
-			(at 163.9728 149.86 0)
+			(at 163.9728 152.4 0)
 			(effects
 				(font
@@
 	(global_label "Fetch"
 		(shape output)
-		(at 153.67 144.78 0)
+		(at 153.67 147.32 0)
 		(fields_autoplaced yes)
 		(effects
@@
 		)
 		(property "Intersheetrefs" "${INTERSHEET_REFS}"
-			(at 161.7957 144.78 0)
+			(at 161.7957 147.32 0)
 			(effects
 				(font
@@
 	(global_label "WB"
 		(shape output)
-		(at 153.67 152.4 0)
+		(at 153.67 144.78 0)
 		(fields_autoplaced yes)
 		(effects
@@
 		)
 		(property "Intersheetrefs" "${INTERSHEET_REFS}"
-			(at 159.3766 152.4 0)
+			(at 159.3766 144.78 0)
 			(effects
 				(font
@@
 		(lib_name "LED_1")
 		(lib_id "Device:LED")
-		(at 124.46 157.48 90)
+		(at 133.35 163.83 90)
 		(unit 1)
 		(exclude_from_sim no)
@@
 		(fields_autoplaced yes)
 		(property "Reference" "D41"
-			(at 128.27 157.7974 90)
+			(at 137.16 164.1474 90)
 			(effects
 				(font
@@
 		)
 		(property "Value" "LED"
-			(at 128.27 160.3374 90)
+			(at 137.16 166.6874 90)
 			(effects
 				(font
@@
 		)
 		(property "Footprint" "LED_THT:LED_D3.0mm_Clear"
-			(at 124.46 157.48 0)
+			(at 133.35 163.83 0)
 			(effects
 				(font
@@
 		)
 		(property "Datasheet" "~"
-			(at 124.46 157.48 0)
+			(at 133.35 163.83 0)
 			(effects
 				(font
@@
 		)
 		(property "Description" "Light emitting diode"
-			(at 124.46 157.48 0)
+			(at 133.35 163.83 0)
 			(effects
 				(font
@@
 		)
 		(property "Sim.Pins" "1=K 2=A"
-			(at 124.46 157.48 0)
+			(at 133.35 163.83 0)
 			(effects
 				(font
@@
 		(lib_name "LED_1")
 		(lib_id "Device:LED")
-		(at 133.35 163.83 90)
+		(at 140.97 157.48 90)
 		(unit 1)
 		(exclude_from_sim no)
@@
 		(fields_autoplaced yes)
 		(property "Reference" "D40"
-			(at 137.16 164.1474 90)
+			(at 144.78 157.7974 90)
 			(effects
 				(font
@@
 		)
 		(property "Value" "LED"
-			(at 137.16 166.6874 90)
+			(at 144.78 160.3374 90)
 			(effects
 				(font
@@
 		)
 		(property "Footprint" "LED_THT:LED_D3.0mm_Clear"
-			(at 133.35 163.83 0)
+			(at 140.97 157.48 0)
 			(effects
 				(font
@@
 		)
 		(property "Datasheet" "~"
-			(at 133.35 163.83 0)
+			(at 140.97 157.48 0)
 			(effects
 				(font
@@
 		)
 		(property "Description" "Light emitting diode"
-			(at 133.35 163.83 0)
+			(at 140.97 157.48 0)
 			(effects
 				(font
@@
 		)
 		(property "Sim.Pins" "1=K 2=A"
-			(at 133.35 163.83 0)
+			(at 140.97 157.48 0)
 			(effects
 				(font
@@
 		(lib_name "LED_1")
 		(lib_id "Device:LED")
-		(at 149.86 163.83 90)
+		(at 124.46 157.48 90)
 		(unit 1)
 		(exclude_from_sim no)
@@
 		(fields_autoplaced yes)
 		(property "Reference" "D38"
-			(at 153.67 164.1474 90)
+			(at 128.27 157.7974 90)
 			(effects
 				(font
@@
 		)
 		(property "Value" "LED"
-			(at 153.67 166.6874 90)
+			(at 128.27 160.3374 90)
 			(effects
 				(font
@@
 		)
 		(property "Footprint" "LED_THT:LED_D3.0mm_Clear"
-			(at 149.86 163.83 0)
+			(at 124.46 157.48 0)
 			(effects
 				(font
@@
 		)
 		(property "Datasheet" "~"
-			(at 149.86 163.83 0)
+			(at 124.46 157.48 0)
 			(effects
 				(font
@@
 		)
 		(property "Description" "Light emitting diode"
-			(at 149.86 163.83 0)
+			(at 124.46 157.48 0)
 			(effects
 				(font
@@
 		)
 		(property "Sim.Pins" "1=K 2=A"
-			(at 149.86 163.83 0)
+			(at 124.46 157.48 0)
 			(effects
 				(font
@@
 		(lib_name "LED_1")
 		(lib_id "Device:LED")
-		(at 140.97 157.48 90)
+		(at 149.86 163.83 90)
 		(unit 1)
 		(exclude_from_sim no)
@@
 		(fields_autoplaced yes)
 		(property "Reference" "D39"
-			(at 144.78 157.7974 90)
+			(at 153.67 164.1474 90)
 			(effects
 				(font
@@
 		)
 		(property "Value" "LED"
-			(at 144.78 160.3374 90)
+			(at 153.67 166.6874 90)
 			(effects
 				(font
@@
 		)
 		(property "Footprint" "LED_THT:LED_D3.0mm_Clear"
-			(at 140.97 157.48 0)
+			(at 149.86 163.83 0)
 			(effects
 				(font
@@
 		)
 		(property "Datasheet" "~"
-			(at 140.97 157.48 0)
+			(at 149.86 163.83 0)
 			(effects
 				(font
@@
 		)
 		(property "Description" "Light emitting diode"
-			(at 140.97 157.48 0)
+			(at 149.86 163.83 0)
 			(effects
 				(font
@@
 		)
 		(property "Sim.Pins" "1=K 2=A"
-			(at 140.97 157.48 0)
+			(at 149.86 163.83 0)
 			(effects
 				(font

Commit message: ver1: ROM_ALU_Decoderの配線を修正
ジャンクション位置と配線経路の見直し(部品・ラベルの増減なし)。
.kicad_pro はKiCADが書き戻した設定差分。

Co-Authored-By: Claude Opus 5 <noreply@anthropic.com>
Connections:
- net GND: no longer IC9.9 (~PE)
- net VDD: now also IC9.9 (~PE)
Changed lines of the file:
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@@
-	)
-	(junction
-		(at 41.91 161.29)
-		(diameter 0)
-		(color 0 0 0 0)
 	)
 	(junction
@@
 	(junction
 		(at 212.09 86.36)
+		(diameter 0)
+		(color 0 0 0 0)
+	)
+	(junction
+		(at 73.66 157.48)
 		(diameter 0)
 		(color 0 0 0 0)
@@
 	(wire
 		(pts
-			(xy 73.66 154.94) (xy 73.66 167.64)
+			(xy 73.66 154.94) (xy 73.66 157.48)
 		)
 		(stroke
@@
 	(wire
 		(pts
-			(xy 41.91 157.48) (xy 41.91 161.29)
+			(xy 41.91 157.48) (xy 41.91 163.83)
 		)
 		(stroke
@@
 	(wire
 		(pts
-			(xy 41.91 161.29) (xy 41.91 163.83)
-		)
-		(stroke
-			(width 0)
-			(type default)
-		)
-	)
-	(wire
-		(pts
 			(xy 107.95 132.08) (xy 107.95 139.7)
 		)
@@
 	(wire
 		(pts
+			(xy 73.66 157.48) (xy 73.66 167.64)
+		)
+		(stroke
+			(width 0)
+			(type default)
+		)
+	)
+	(wire
+		(pts
 			(xy 261.62 195.58) (xy 270.51 195.58)
 		)
@@
 	(wire
 		(pts
-			(xy 71.12 157.48) (xy 72.39 157.48)
+			(xy 71.12 157.48) (xy 73.66 157.48)
 		)
 		(stroke
@@
 	(wire
 		(pts
-			(xy 72.39 161.29) (xy 41.91 161.29)
-		)
-		(stroke
-			(width 0)
-			(type default)
-		)
-	)
-	(wire
-		(pts
 			(xy 107.95 168.91) (xy 107.95 170.18)
 		)
@@
 		)
 		(stroke
-			(width 0)
-			(type default)
-		)
-	)
-	(wire
-		(pts
-			(xy 72.39 157.48) (xy 72.39 161.29)
-		)
-		(stroke
