File: ver2/hardware/TB04addr8bit/ROM_ALU.kicad_sch (KiCad schematic)
At the start: 27 parts, among them IC9 74HC161N, U10 74LS08, U11 74LS273, U14 74HC238, U20 74HC273, U21 74HC74, U22 74HC273, U24 28C256, U5 28C256

Commit message: ver2: PC_mAddr中心に回路図の配線を更新
7/18のコミット以降の結線作業を反映。部品・ラベルの増減はなく、
配線(wire)とジャンクションの変更のみ。
- PC_mAddr.kicad_sch: 配線36箇所
- sp.kicad_sch / ROM_ALU.kicad_sch / ルートシート: 数箇所ずつ
- TB04addr8bit.kicad_pro: KiCAD 10がERC重要度・last_pathsの
  既定値を追記したもの(設定の書き戻しで設計内容の変化ではない)

なおこの状態のネットリストを ai-review で出力してレビュー済み。
要修正5件と残作業は ver2/DEVLOG.md(2026-08-10)に記録した(未着手)。

Co-Authored-By: Claude Opus 5 <noreply@anthropic.com>
Connections:
- net GND: no longer IC9.9 (~PE)
- net VDD: now also IC9.9 (~PE)
Changed lines of the file:
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@@
+	)
+	(junction
+		(at 92.71 231.14)
+		(diameter 0)
+		(color 0 0 0 0)
 	)
 	(junction
@@
 	(junction
 		(at 330.2 203.2)
-		(diameter 0)
-		(color 0 0 0 0)
-	)
-	(junction
-		(at 60.96 234.95)
 		(diameter 0)
 		(color 0 0 0 0)
@@
 	(wire
 		(pts
-			(xy 92.71 228.6) (xy 92.71 241.3)
+			(xy 92.71 228.6) (xy 92.71 231.14)
 		)
 		(stroke
@@
 	(wire
 		(pts
-			(xy 60.96 231.14) (xy 60.96 234.95)
-		)
-		(stroke
-			(width 0)
-			(type default)
-		)
-	)
-	(wire
-		(pts
 			(xy 241.3 129.54) (xy 245.11 129.54)
 		)
@@
 	(wire
 		(pts
+			(xy 92.71 231.14) (xy 92.71 241.3)
+		)
+		(stroke
+			(width 0)
+			(type default)
+		)
+	)
+	(wire
+		(pts
 			(xy 330.2 213.36) (xy 331.47 213.36)
 		)
@@
 	(wire
 		(pts
-			(xy 60.96 234.95) (xy 60.96 237.49)
+			(xy 60.96 231.14) (xy 60.96 237.49)
 		)
 		(stroke
@@
 	(wire
 		(pts
-			(xy 90.17 231.14) (xy 91.44 231.14)
+			(xy 90.17 231.14) (xy 92.71 231.14)
 		)
 		(stroke
@@
 	(wire
 		(pts
-			(xy 91.44 234.95) (xy 60.96 234.95)
-		)
-		(stroke
-			(width 0)
-			(type default)
-		)
-	)
-	(wire
-		(pts
 			(xy 247.65 87.63) (xy 247.65 99.06)
 		)
@@
 		)
 		(stroke
-			(width 0)
-			(type default)
-		)
-	)
-	(wire
-		(pts
-			(xy 91.44 231.14) (xy 91.44 234.95)
-		)
-		(stroke
