File: ver2/hardware/TB04addr8bit/ALU.kicad_sch (KiCad schematic)
At the start: 23 parts

Commit message: ver2: 回路図の要修正5件を修正しアノテーションを掛け直し
- 74HC193(旧U39/新U38)の~CO・~BOをVDD直結から開放に(出力短絡の回避)
- 電源未接続だった4IC(74HC00/74LS32/74AHC04/74LS08)にVCC/GNDを配線
  し、バイパスコンデンサ0.1u×4を追加
- ネット名 Decord を DCR に統一(デコーダ制御信号のラッチ不成立を解消)
- PC_LAOD の綴りを PC_LOAD に修正
- 書込デコーダ138の入力を OPR8-10 から sel_a0-2 へ付け替え
  (LD Ri,[Im8] が別レジスタに書く不具合の解消)
- ver1基板由来だった参照記号をアノテーション掛け直しで整理
  (部品216個・名前付きネット146本とも掛け直し前後で一致、ERCも同数)
Parts:
- renumbered D18 to D42, D20 to D43, D51 to D44, D53 to D45, D31 to D46, D33 to D47, D45 to D48, D47 to D49, D35 to D50, D37 to D51, D17 to D52, D19 to D53, D50 to D54, D52 to D55, D30 to D56, D32 to D57, D44 to D58, D46 to D59, D34 to D60, D36 to D61, RN3 to RN6, RN9 to RN7, RN7 to RN8
Changed lines of the file:
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@@
 		(dnp no)
 		(fields_autoplaced yes)
-		(property "Reference" "D34"
+		(property "Reference" "D60"
 			(at 237.49 112.0774 90)
 			(show_name no)
@@
 			(project "TB04addr8bit"
 				(path "/d176c79b-dced-4d01-bcec-7dfd676fcfc2/8128481a-591d-4f1a-bdfd-fb80959a87d7"
-					(reference "D34")
+					(reference "D60")
 					(unit 1)
 				)
@@
 		(dnp no)
 		(fields_autoplaced yes)
-		(property "Reference" "D47"
+		(property "Reference" "D49"
 			(at 96.52 105.7274 90)
 			(show_name no)
@@
 			(project "TB04addr8bit"
 				(path "/d176c79b-dced-4d01-bcec-7dfd676fcfc2/8128481a-591d-4f1a-bdfd-fb80959a87d7"
-					(reference "D47")
+					(reference "D49")
 					(unit 1)
 				)
@@
 		(dnp no)
 		(fields_autoplaced yes)
-		(property "Reference" "D53"
+		(property "Reference" "D45"
 			(at 147.32 104.4574 90)
 			(show_name no)
@@
 			(project "TB04addr8bit"
 				(path "/d176c79b-dced-4d01-bcec-7dfd676fcfc2/8128481a-591d-4f1a-bdfd-fb80959a87d7"
-					(reference "D53")
+					(reference "D45")
 					(unit 1)
 				)
@@
 		(dnp no)
 		(fields_autoplaced yes)
-		(property "Reference" "D20"
+		(property "Reference" "D43"
 			(at 330.2 101.9174 90)
 			(show_name no)
@@
 			(project "TB04addr8bit"
 				(path "/d176c79b-dced-4d01-bcec-7dfd676fcfc2/8128481a-591d-4f1a-bdfd-fb80959a87d7"
-					(reference "D20")
+					(reference "D43")
 					(unit 1)
 				)
@@
 		(dnp no)
 		(fields_autoplaced yes)
-		(property "Reference" "D50"
+		(property "Reference" "D54"
 			(at 121.92 110.8074 90)
 			(show_name no)
@@
 			(project "TB04addr8bit"
 				(path "/d176c79b-dced-4d01-bcec-7dfd676fcfc2/8128481a-591d-4f1a-bdfd-fb80959a87d7"
-					(reference "D50")
+					(reference "D54")
 					(unit 1)
 				)
@@
 		(dnp no)
 		(fields_autoplaced yes)
-		(property "Reference" "D33"
+		(property "Reference" "D47"
 			(at 203.2 104.4574 90)
 			(show_name no)
@@
 			(project "TB04addr8bit"
 				(path "/d176c79b-dced-4d01-bcec-7dfd676fcfc2/8128481a-591d-4f1a-bdfd-fb80959a87d7"
-					(reference "D33")
+					(reference "D47")
 					(unit 1)
 				)
@@
 		(dnp no)
 		(fields_autoplaced yes)
-		(property "Reference" "D35"
+		(property "Reference" "D50"
 			(at 246.38 105.7274 90)
 			(show_name no)
@@
 			(project "TB04addr8bit"
 				(path "/d176c79b-dced-4d01-bcec-7dfd676fcfc2/8128481a-591d-4f1a-bdfd-fb80959a87d7"
-					(reference "D35")
+					(reference "D50")
 					(unit 1)
 				)
@@
 		(dnp no)
 		(fields_autoplaced yes)
-		(property "Reference" "RN3"
+		(property "Reference" "RN6"
 			(at 323.85 139.4459 0)
 			(show_name no)
@@
 			(project "TB04addr8bit"
 				(path "/d176c79b-dced-4d01-bcec-7dfd676fcfc2/8128481a-591d-4f1a-bdfd-fb80959a87d7"
-					(reference "RN3")
+					(reference "RN6")
 					(unit 1)
 				)
@@
 		(dnp no)
 		(fields_autoplaced yes)
-		(property "Reference" "D19"
+		(property "Reference" "D53"
 			(at 321.31 108.2674 90)
 			(show_name no)
@@
 			(project "TB04addr8bit"
 				(path "/d176c79b-dced-4d01-bcec-7dfd676fcfc2/8128481a-591d-4f1a-bdfd-fb80959a87d7"
-					(reference "D19")
+					(reference "D53")
 					(unit 1)
 				)
@@
 		(dnp no)
 		(fields_autoplaced yes)
-		(property "Reference" "D18"
+		(property "Reference" "D42"
 			(at 313.69 101.9174 90)
 			(show_name no)
@@
 			(project "TB04addr8bit"
 				(path "/d176c79b-dced-4d01-bcec-7dfd676fcfc2/8128481a-591d-4f1a-bdfd-fb80959a87d7"
-					(reference "D18")
+					(reference "D42")
 					(unit 1)
 				)
@@
 		(dnp no)
 		(fields_autoplaced yes)
-		(property "Reference" "D17"
+		(property "Reference" "D52"
 			(at 304.8 108.2674 90)
 			(show_name no)
@@
 			(project "TB04addr8bit"
 				(path "/d176c79b-dced-4d01-bcec-7dfd676fcfc2/8128481a-591d-4f1a-bdfd-fb80959a87d7"
-					(reference "D17")
+					(reference "D52")
 					(unit 1)
 				)
@@
 		(dnp no)
 		(fields_autoplaced yes)
-		(property "Reference" "RN9"
+		(property "Reference" "RN7"
 			(at 102.87 148.3359 0)
 			(show_name no)
@@
 			(project "TB04addr8bit"
 				(path "/d176c79b-dced-4d01-bcec-7dfd676fcfc2/8128481a-591d-4f1a-bdfd-fb80959a87d7"
-					(reference "RN9")
+					(reference "RN7")
 					(unit 1)
 				)
@@
 		(dnp no)
 		(fields_autoplaced yes)
-		(property "Reference" "D36"
+		(property "Reference" "D61"
 			(at 254 112.0774 90)
 			(show_name no)
@@
 			(project "TB04addr8bit"
 				(path "/d176c79b-dced-4d01-bcec-7dfd676fcfc2/8128481a-591d-4f1a-bdfd-fb80959a87d7"
-					(reference "D36")
+					(reference "D61")
 					(unit 1)
 				)
@@
 		(dnp no)
 		(fields_autoplaced yes)
-		(property "Reference" "RN7"
+		(property "Reference" "RN8"
 			(at 208.28 157.2259 0)
 			(show_name no)
@@
 			(project "TB04addr8bit"
 				(path "/d176c79b-dced-4d01-bcec-7dfd676fcfc2/8128481a-591d-4f1a-bdfd-fb80959a87d7"
-					(reference "RN7")
+					(reference "RN8")
 					(unit 1)
 				)
@@
 		(dnp no)
 		(fields_autoplaced yes)
-		(property "Reference" "D32"
+		(property "Reference" "D57"
 			(at 194.31 110.8074 90)
 			(show_name no)
@@
 			(project "TB04addr8bit"
 				(path "/d176c79b-dced-4d01-bcec-7dfd676fcfc2/8128481a-591d-4f1a-bdfd-fb80959a87d7"
-					(reference "D32")
+					(reference "D57")
 					(unit 1)
 				)
@@
 		(dnp no)
 		(fields_autoplaced yes)
-		(property "Reference" "D44"
+		(property "Reference" "D58"
 			(at 71.12 112.0774 90)
 			(show_name no)
@@
 			(project "TB04addr8bit"
 				(path "/d176c79b-dced-4d01-bcec-7dfd676fcfc2/8128481a-591d-4f1a-bdfd-fb80959a87d7"
-					(reference "D44")
+					(reference "D58")
 					(unit 1)
 				)
@@
 		(dnp no)
 		(fields_autoplaced yes)
-		(property "Reference" "D37"
+		(property "Reference" "D51"
 			(at 262.89 105.7274 90)
 			(show_name no)
@@
 			(project "TB04addr8bit"
 				(path "/d176c79b-dced-4d01-bcec-7dfd676fcfc2/8128481a-591d-4f1a-bdfd-fb80959a87d7"
-					(reference "D37")
+					(reference "D51")
 					(unit 1)
 				)
@@
 		(dnp no)
 		(fields_autoplaced yes)
-		(property "Reference" "D45"
+		(property "Reference" "D48"
 			(at 80.01 105.7274 90)
 			(show_name no)
@@
 			(project "TB04addr8bit"
 				(path "/d176c79b-dced-4d01-bcec-7dfd676fcfc2/8128481a-591d-4f1a-bdfd-fb80959a87d7"
-					(reference "D45")
+					(reference "D48")
 					(unit 1)
 				)
@@
 		(dnp no)
 		(fields_autoplaced yes)
-		(property "Reference" "D51"
+		(property "Reference" "D44"
 			(at 130.81 104.4574 90)
 			(show_name no)
@@
 			(project "TB04addr8bit"
 				(path "/d176c79b-dced-4d01-bcec-7dfd676fcfc2/8128481a-591d-4f1a-bdfd-fb80959a87d7"
-					(reference "D51")
+					(reference "D44")
 					(unit 1)
 				)
@@
 		(dnp no)
 		(fields_autoplaced yes)
-		(property "Reference" "D52"
+		(property "Reference" "D55"
 			(at 138.43 110.8074 90)
 			(show_name no)
@@
 			(project "TB04addr8bit"
 				(path "/d176c79b-dced-4d01-bcec-7dfd676fcfc2/8128481a-591d-4f1a-bdfd-fb80959a87d7"
-					(reference "D52")
+					(reference "D55")
 					(unit 1)
 				)
@@
 		(dnp no)
 		(fields_autoplaced yes)
-		(property "Reference" "#PWR0101"
+		(property "Reference" "#PWR0118"
 			(at 105.41 165.1 0)
 			(hide yes)
@@
 			(project "TB04addr8bit"
 				(path "/d176c79b-dced-4d01-bcec-7dfd676fcfc2/8128481a-591d-4f1a-bdfd-fb80959a87d7"
-					(reference "#PWR0101")
+					(reference "#PWR0118")
 					(unit 1)
 				)
@@
 		(dnp no)
 		(fields_autoplaced yes)
-		(property "Reference" "D46"
+		(property "Reference" "D59"
 			(at 87.63 112.0774 90)
 			(show_name no)
@@
 			(project "TB04addr8bit"
 				(path "/d176c79b-dced-4d01-bcec-7dfd676fcfc2/8128481a-591d-4f1a-bdfd-fb80959a87d7"
-					(reference "D46")
+					(reference "D59")
 					(unit 1)
 				)
@@
 		(dnp no)
 		(fields_autoplaced yes)
-		(property "Reference" "#PWR0103"
+		(property "Reference" "#PWR0117"
 			(at 326.39 154.94 0)
 			(hide yes)
@@
 			(project "TB04addr8bit"
 				(path "/d176c79b-dced-4d01-bcec-7dfd676fcfc2/8128481a-591d-4f1a-bdfd-fb80959a87d7"
-					(reference "#PWR0103")
+					(reference "#PWR0117")
 					(unit 1)
 				)
@@
 		(dnp no)
 		(fields_autoplaced yes)
-		(property "Reference" "D30"
+		(property "Reference" "D56"
 			(at 177.8 110.8074 90)
 			(show_name no)
@@
 			(project "TB04addr8bit"
 				(path "/d176c79b-dced-4d01-bcec-7dfd676fcfc2/8128481a-591d-4f1a-bdfd-fb80959a87d7"
-					(reference "D30")
+					(reference "D56")
 					(unit 1)
 				)
@@
 		(dnp no)
 		(fields_autoplaced yes)
-		(property "Reference" "D31"
+		(property "Reference" "D46"
 			(at 186.69 104.4574 90)
 			(show_name no)
@@
 			(project "TB04addr8bit"
 				(path "/d176c79b-dced-4d01-bcec-7dfd676fcfc2/8128481a-591d-4f1a-bdfd-fb80959a87d7"
-					(reference "D31")
+					(reference "D46")
 					(unit 1)
 				)
@@
 		(dnp no)
 		(fields_autoplaced yes)
-		(property "Reference" "#PWR0102"
+		(property "Reference" "#PWR0119"
 			(at 210.82 172.72 0)
 			(hide yes)
@@
 			(project "TB04addr8bit"
 				(path "/d176c79b-dced-4d01-bcec-7dfd676fcfc2/8128481a-591d-4f1a-bdfd-fb80959a87d7"
-					(reference "#PWR0102")
-					(unit 1)
-				)
+					(reference "#PWR0119")
+					(unit 1)
+				)
