File: ver2/hardware/TB04addr8bit/clk_rst.kicad_sch (KiCad schematic)
At the start: 30 parts, among them SW4 SW_DIP_x04, SW5 SW_SPDT, SW6 SW_Push, SW7 SW_Push, U12 4060, U17 74HC14, Y1 32.768KHz

Commit message: ver2: 回路図の要修正5件を修正しアノテーションを掛け直し
- 74HC193(旧U39/新U38)の~CO・~BOをVDD直結から開放に(出力短絡の回避)
- 電源未接続だった4IC(74HC00/74LS32/74AHC04/74LS08)にVCC/GNDを配線
  し、バイパスコンデンサ0.1u×4を追加
- ネット名 Decord を DCR に統一(デコーダ制御信号のラッチ不成立を解消)
- PC_LAOD の綴りを PC_LOAD に修正
- 書込デコーダ138の入力を OPR8-10 から sel_a0-2 へ付け替え
  (LD Ri,[Im8] が別レジスタに書く不具合の解消)
- ver1基板由来だった参照記号をアノテーション掛け直しで整理
  (部品216個・名前付きネット146本とも掛け直し前後で一致、ERCも同数)
Parts:
- renumbered C32 to C30, C33 to C31, C22 to C32, C27 to C33, C21 to C34, C29 to C35, D49 to D34, D48 to D35, H3 to H2, H4 to H3, H2 to H4, R25 to R10, R29 to R11, R28 to R12, R1 to R13, R2 to R14, R30 to R4, R31 to R5, R26 to R6, R24 to R7, R23 to R8, R27 to R9, SW6 to SW2, SW5 to SW3, SW7 to SW4, SW4 to SW5, U17 to U18, U12 to U19

Commit message: ver2: クロック選択をロータリースイッチ化、PCの桁上げ配線に着手
- クロック選択をDIP4連から1回路9接点ロータリー(SW7)へ変更
  左端=マニュアル、以降Q13/Q12/Q10/Q9/Q8/Q6/Q5/Q4の順で
  1→2→8→16→32→128→256→512命令/秒と右回りに高速化
  DIPのコモン短絡問題が構造的に解消。コモンに100Kプルダウン(R17)を追加し
  切替時の浮きを防止。取付ピン(MP)はGNDへ
- PC_mAddr: CNTABLラベルを廃止し、161×4のCEPを共通ネットにまとめ
  IC10のTC→IC9のCET、IC12のTC→IC11のCETで桁上げを接続(作業中)
Parts:
- removed SW3: SW_SPDT, Library:sw_slide, symbol Switch:SW_SPDT
- removed SW5: SW_DIP_x04, Button_Switch_THT:SW_DIP_SPSTx04_Slide_9.78x12.34mm_W7.62mm_P2.54mm, symbol Switch:SW_DIP_x04
- added R17: 100K, symbol Device:R
- added SW7: SW_Rotary_1x9_MP, symbol Switch:SW_Rotary_1x9_MP
Connections:
- net GND: now also R17.2, SW7.MP
- net at R12.1, U18.9: now also R17.1, SW7.10
- net at U19.1 (Q12): now also SW7.3
- net at U19.13 (Q9): now also SW7.5
- net at U19.14 (Q8): now also SW7.6
- net at U19.15 (Q10): now also SW7.4
- net at U19.2 (Q13): now also SW7.2
- net at U19.4 (Q6): now also SW7.7
- net at U19.5 (Q5): now also SW7.8
- net at U19.7 (Q4): now also SW7.9
- net at R8.2: now also SW7.1
- no-connect marks 9 -> 5
Other:
- note added: "Fast"
- note added: "Slow"
- moved on the sheet: C30, D35, R12, R4, R6, R7, R8, SW2, U18C, U18D
