File: ver2/hardware/TB04addr8bit/AddrDecord.kicad_sch (KiCad schematic)
At the start: 6 parts, among them U31 74LS08, U32 74AHC04, U36 74LS08

Commit message: ver2: 回路図の要修正5件を修正しアノテーションを掛け直し
- 74HC193(旧U39/新U38)の~CO・~BOをVDD直結から開放に(出力短絡の回避)
- 電源未接続だった4IC(74HC00/74LS32/74AHC04/74LS08)にVCC/GNDを配線
  し、バイパスコンデンサ0.1u×4を追加
- ネット名 Decord を DCR に統一(デコーダ制御信号のラッチ不成立を解消)
- PC_LAOD の綴りを PC_LOAD に修正
- 書込デコーダ138の入力を OPR8-10 から sel_a0-2 へ付け替え
  (LD Ri,[Im8] が別レジスタに書く不具合の解消)
- ver1基板由来だった参照記号をアノテーション掛け直しで整理
  (部品216個・名前付きネット146本とも掛け直し前後で一致、ERCも同数)
Parts:
- renumbered C45 to C57, C47 to C58, C48 to C59, U32 to U1, U31 to U39, U36 to U40
Changed lines of the file:
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@@
 		(dnp no)
 		(fields_autoplaced yes)
-		(property "Reference" "U36"
+		(property "Reference" "U40"
 			(at 93.9717 130.81 0)
 			(show_name no)
@@
 			(project "TB04addr8bit"
 				(path "/d176c79b-dced-4d01-bcec-7dfd676fcfc2/5966379b-e25d-4be9-810c-b95428770124"
-					(reference "U36")
+					(reference "U40")
 					(unit 4)
 				)
@@
 		(dnp no)
 		(fields_autoplaced yes)
-		(property "Reference" "U36"
+		(property "Reference" "U40"
 			(at 93.9717 113.03 0)
 			(show_name no)
@@
 			(project "TB04addr8bit"
 				(path "/d176c79b-dced-4d01-bcec-7dfd676fcfc2/5966379b-e25d-4be9-810c-b95428770124"
-					(reference "U36")
+					(reference "U40")
 					(unit 3)
 				)
@@
 		(dnp no)
 		(fields_autoplaced yes)
-		(property "Reference" "U32"
+		(property "Reference" "U1"
 			(at 76.2 115.57 0)
 			(show_name no)
@@
 			(project "TB04addr8bit"
 				(path "/d176c79b-dced-4d01-bcec-7dfd676fcfc2/5966379b-e25d-4be9-810c-b95428770124"
-					(reference "U32")
+					(reference "U1")
 					(unit 3)
 				)
@@
 		(dnp no)
 		(fields_autoplaced yes)
-		(property "Reference" "C48"
+		(property "Reference" "C59"
 			(at 257.81 82.5499 0)
 			(show_name no)
@@
 			(project "TB04addr8bit"
 				(path "/d176c79b-dced-4d01-bcec-7dfd676fcfc2/5966379b-e25d-4be9-810c-b95428770124"
-					(reference "C48")
+					(reference "C59")
 					(unit 1)
 				)
@@
 		(dnp no)
 		(fields_autoplaced yes)
-		(property "Reference" "U32"
+		(property "Reference" "U1"
 			(at 93.98 78.74 0)
 			(show_name no)
@@
 			(project "TB04addr8bit"
 				(path "/d176c79b-dced-4d01-bcec-7dfd676fcfc2/5966379b-e25d-4be9-810c-b95428770124"
-					(reference "U32")
+					(reference "U1")
 					(unit 1)
 				)
@@
 		(dnp no)
 		(fields_autoplaced yes)
-		(property "Reference" "U32"
+		(property "Reference" "U1"
 			(at 226.06 121.9199 0)
 			(show_name no)
@@
 			(project "TB04addr8bit"
 				(path "/d176c79b-dced-4d01-bcec-7dfd676fcfc2/5966379b-e25d-4be9-810c-b95428770124"
-					(reference "U32")
+					(reference "U1")
 					(unit 7)
 				)
@@
 		(dnp no)
 		(fields_autoplaced yes)
-		(property "Reference" "U32"
+		(property "Reference" "U1"
 			(at 76.2 133.35 0)
 			(show_name no)
@@
 			(project "TB04addr8bit"
 				(path "/d176c79b-dced-4d01-bcec-7dfd676fcfc2/5966379b-e25d-4be9-810c-b95428770124"
-					(reference "U32")
+					(reference "U1")
 					(unit 4)
 				)
@@
 		(dnp no)
 		(fields_autoplaced yes)
-		(property "Reference" "#PWR010"
+		(property "Reference" "#PWR0132"
 			(at 231.14 97.79 0)
 			(hide yes)
@@
 			(project "TB04addr8bit"
 				(path "/d176c79b-dced-4d01-bcec-7dfd676fcfc2/5966379b-e25d-4be9-810c-b95428770124"
-					(reference "#PWR010")
+					(reference "#PWR0132")
 					(unit 1)
 				)
@@
 		(dnp no)
 		(fields_autoplaced yes)
-		(property "Reference" "U36"
+		(property "Reference" "U40"
 			(at 93.9717 93.98 0)
 			(show_name no)
@@
 			(project "TB04addr8bit"
 				(path "/d176c79b-dced-4d01-bcec-7dfd676fcfc2/5966379b-e25d-4be9-810c-b95428770124"
-					(reference "U36")
+					(reference "U40")
 					(unit 2)
 				)
@@
 		(dnp no)
 		(fields_autoplaced yes)
-		(property "Reference" "U32"
+		(property "Reference" "U1"
 			(at 74.93 96.52 0)
 			(show_name no)
@@
 			(project "TB04addr8bit"
 				(path "/d176c79b-dced-4d01-bcec-7dfd676fcfc2/5966379b-e25d-4be9-810c-b95428770124"
-					(reference "U32")
+					(reference "U1")
 					(unit 2)
 				)
@@
 		(dnp no)
 		(fields_autoplaced yes)
-		(property "Reference" "#PWR09"
+		(property "Reference" "#PWR0133"
 			(at 199.39 148.59 0)
 			(hide yes)
@@
 			(project "TB04addr8bit"
 				(path "/d176c79b-dced-4d01-bcec-7dfd676fcfc2/5966379b-e25d-4be9-810c-b95428770124"
-					(reference "#PWR09")
+					(reference "#PWR0133")
 					(unit 1)
 				)
@@
 		(dnp no)
 		(fields_autoplaced yes)
-		(property "Reference" "C47"
+		(property "Reference" "C58"
 			(at 246.38 82.5499 0)
 			(show_name no)
@@
 			(project "TB04addr8bit"
 				(path "/d176c79b-dced-4d01-bcec-7dfd676fcfc2/5966379b-e25d-4be9-810c-b95428770124"
-					(reference "C47")
+					(reference "C58")
 					(unit 1)
 				)
@@
 		(dnp no)
 		(fields_autoplaced yes)
-		(property "Reference" "U31"
+		(property "Reference" "U39"
 			(at 88.8917 57.15 0)
 			(show_name no)
@@
 			(project "TB04addr8bit"
 				(path "/d176c79b-dced-4d01-bcec-7dfd676fcfc2/5966379b-e25d-4be9-810c-b95428770124"
-					(reference "U31")
+					(reference "U39")
 					(unit 2)
 				)
@@
 		(dnp no)
 		(fields_autoplaced yes)
-		(property "Reference" "U31"
+		(property "Reference" "U39"
 			(at 140.9617 62.23 0)
 			(show_name no)
@@
 			(project "TB04addr8bit"
 				(path "/d176c79b-dced-4d01-bcec-7dfd676fcfc2/5966379b-e25d-4be9-810c-b95428770124"
-					(reference "U31")
+					(reference "U39")
 					(unit 4)
 				)
@@
 		(dnp no)
 		(fields_autoplaced yes)
-		(property "Reference" "U31"
+		(property "Reference" "U39"
 			(at 114.2917 54.61 0)
 			(show_name no)
@@
 			(project "TB04addr8bit"
 				(path "/d176c79b-dced-4d01-bcec-7dfd676fcfc2/5966379b-e25d-4be9-810c-b95428770124"
-					(reference "U31")
+					(reference "U39")
 					(unit 3)
 				)
@@
 		(dnp no)
 		(fields_autoplaced yes)
-		(property "Reference" "C45"
+		(property "Reference" "C57"
 			(at 234.95 82.5499 0)
 			(show_name no)
@@
 			(project "TB04addr8bit"
 				(path "/d176c79b-dced-4d01-bcec-7dfd676fcfc2/5966379b-e25d-4be9-810c-b95428770124"
-					(reference "C45")
+					(reference "C57")
 					(unit 1)
 				)
@@
 		(dnp no)
 		(fields_autoplaced yes)
-		(property "Reference" "U36"
+		(property "Reference" "U40"
 			(at 163.8217 71.12 0)
 			(show_name no)
@@
 			(project "TB04addr8bit"
 				(path "/d176c79b-dced-4d01-bcec-7dfd676fcfc2/5966379b-e25d-4be9-810c-b95428770124"
-					(reference "U36")
+					(reference "U40")
 					(unit 1)
 				)
@@
 		(dnp no)
 		(fields_autoplaced yes)
-		(property "Reference" "U36"
+		(property "Reference" "U40"
 			(at 247.65 121.9199 0)
 			(show_name no)
@@
 			(project "TB04addr8bit"
 				(path "/d176c79b-dced-4d01-bcec-7dfd676fcfc2/5966379b-e25d-4be9-810c-b95428770124"
-					(reference "U36")
+					(reference "U40")
 					(unit 5)
 				)
@@
 		(dnp no)
 		(fields_autoplaced yes)
-		(property "Reference" "U31"
+		(property "Reference" "U39"
 			(at 205.74 121.9199 0)
 			(show_name no)
@@
 			(project "TB04addr8bit"
 				(path "/d176c79b-dced-4d01-bcec-7dfd676fcfc2/5966379b-e25d-4be9-810c-b95428770124"
-					(reference "U31")
+					(reference "U39")
 					(unit 5)
 				)
@@
 		(dnp no)
 		(fields_autoplaced yes)
-		(property "Reference" "U31"
+		(property "Reference" "U39"
 			(at 88.8917 35.56 0)
 			(show_name no)
@@
 			(project "TB04addr8bit"
 				(path "/d176c79b-dced-4d01-bcec-7dfd676fcfc2/5966379b-e25d-4be9-810c-b95428770124"
-					(reference "U31")
+					(reference "U39")
 					(unit 1)
 				)

Commit message: ver2: addrMUXシートを新設、リセット起点をFCH1へ、mAddr専用レジスタを廃止
- addrMUX.kicad_sch を新設。74HC138(U41)で SEL_M からアドレス源の
  イネーブルをワンホット生成し、74HC244×5(U42-U46)を配置
  mAddr用(U43)の入力は byte2ラッチのOPR4-11から直取り
- mAddr専用レジスタ(IC11/IC12)を削除。byte2ラッチが mAddr を兼ねる
  これまで消費先ゼロだった OPR7/OPR11 の浮きも解消
- 74HC238の出力割付を1つ回してリセット起点を EXE から FCH1 へ
  (Y0=FCH1/Y1=FCH2/Y2=DCR/Y3=EXE、相順は不変)
- PCの161はCEPを共通イネーブルに揃え、桁上げをTC->CETで接続

未了: 命令ラッチの取り込みエッジを1相ずらす変更(U20 Cp=FCH2 /
U26 Cp=DCR)。EXE中はアドレスバスがmAddrのため、現状のままでは
EXE->FCH1の境目でROMのアクセスが間に合わない
Other:
- moved on the sheet: C57, C58, C59, U1A, U1B, U1C, U1D, U1G, U39A, U39B, U39C, U39D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
