File: ver2/hardware/TB04_1_alu/TB04_1_alu.kicad_sch (KiCad schematic)
At the start: 11 parts, among them J101 Conn_02x20_Odd_Even, J102 Conn_02x20_Odd_Even, J103 Conn_02x20_Odd_Even, U101 74LS157, U102 74HC138

Commit message: ver2: 制御基板を分割完了・不要シートを整理(基板4分割の3枚目)
TB04_2_ctrl を分割完了。ai-reviewで検証し合格。
- 64信号すべてバスへ引き出し済み、ピン位置は確定表と完全一致
- 署名が変わったのは J101 のみ(USB-C→40ピンバスヘッダ)
- 電源入口は TB04_4_io のみ。他基板はバス1のVDD/GNDから受ける
- 各プロジェクトから未使用シートのファイルを削除

Co-Authored-By: Claude Opus 5 <noreply@anthropic.com>
Connections:
- net OPR0: now also J102.1 (Pin_1); no longer J102.39 (Pin_39)
- net OPR1: now also J102.3 (Pin_3); no longer J102.37 (Pin_37)
- net OPR10: now also J102.13 (Pin_13); no longer J102.15 (Pin_15)
- net OPR2: now also J102.5 (Pin_5); no longer J102.35 (Pin_35)
- net OPR3: now also J102.6 (Pin_6); no longer J102.33 (Pin_33)
- net OPR4: now also J102.7 (Pin_7); no longer J102.31 (Pin_31)
- net OPR5: now also J102.8 (Pin_8); no longer J102.29 (Pin_29)
- net OPR6: now also J102.9 (Pin_9); no longer J102.27 (Pin_27)
- net OPR7: now also J102.10 (Pin_10); no longer J102.25 (Pin_25)
- net OPR8: now also J102.11 (Pin_11); no longer J102.19 (Pin_19)
- net OPR9: now also J102.12 (Pin_12); no longer J102.17 (Pin_17)
- net RegAddrSrc: now also J102.25 (Pin_25); no longer J102.20 (Pin_20)
- net SEL_A: now also J102.19 (Pin_19); no longer J102.3 (Pin_3)
- net SEL_B0: now also J102.20 (Pin_20); no longer J102.1 (Pin_1)
- net SEL_B1: now also J102.22 (Pin_22); no longer J102.24 (Pin_24)
- net SEL_IMM: now also J102.24 (Pin_24); no longer J102.22 (Pin_22)
- net YD0: now also J103.19 (Pin_19); no longer J103.7 (Pin_7)
- net YD1: now also J103.20 (Pin_20); no longer J103.5 (Pin_5)
- net YD2: now also J103.22 (Pin_22); no longer J103.3 (Pin_3)
- net YD3: now also J103.24 (Pin_24); no longer J103.1 (Pin_1)
- net alu_code0: now also J102.15 (Pin_15); no longer J102.11 (Pin_11)
- net alu_code1: now also J102.16 (Pin_16); no longer J102.9 (Pin_9)
- net alu_code2: now also J102.17 (Pin_17); no longer J102.7 (Pin_7)
- net alu_code3: now also J102.18 (Pin_18); no longer J102.5 (Pin_5)
- net carry_in: now also J102.35 (Pin_35); no longer J102.10 (Pin_10)
- net carry_out: now also J102.37 (Pin_37); no longer J102.8 (Pin_8)
- net sel_a2: now also J102.27 (Pin_27); no longer J102.16 (Pin_16)
- net zero_flag: now also J102.39 (Pin_39); no longer J102.6 (Pin_6)
- net ~{Ena_RS01}: now also J102.31 (Pin_31); no longer J102.14 (Pin_14)
- net ~{Enb_RS01}: now also J102.33 (Pin_33); no longer J102.12 (Pin_12)
- net ~{WE}: now also J102.29 (Pin_29); no longer J102.18 (Pin_18)
- net CLK_CPU: now reaches J101.1 (Pin_1)
- net ~{RST}: now reaches J101.7 (Pin_7)
- no-connect marks 41 -> 39
