File: ver2/hardware/基板分割_0825/TB04_S4_addr/TB04_S4_addr.kicad_sch (KiCad schematic)
At the start: 10 parts, among them J101 Conn_02x20_Odd_Even, J102 Conn_02x20_Odd_Even, J103 Conn_02x20_Odd_Even, J104 Conn_02x10_Odd_Even, J105 Conn_02x10_Odd_Even, J106 Conn_02x10_Odd_Even

Commit message: ver2: キャリアに7segIF用2×5コネクタ4個と電源部を実装／全7枚に予備の端子台
- キャリア: J3-J6(2×5)が桁1-4で表と全一致・DIG_*16ネットは2ピン構成
  (isolated_pin_label 16件→0件)、C1/C2/電源LED/端子台を追加
- 入力の2×10はJ1→J2にリナンバー(20ピンの中身は表と一致)
- 7枚とも端子台J1602を1個ずつ追加(pin1=＋/pin2=GNDで向きは全枚統一)
- 署名比較で既存ピンのネット変化は7枚とも0件(吸着なし)

Co-Authored-By: Claude Opus 5 <noreply@anthropic.com>
Parts:
- added J1602: Screw_Terminal_01x02, symbol Connector:Screw_Terminal_01x02
Connections:
- net GND: now also J1602.2 (Pin_2)
- net VDD: now also J1602.1 (Pin_1)
Changed lines of the file:
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@@
 	)
 	(junction
+		(at 157.48 62.23)
+		(diameter 0)
+		(color 0 0 0 0)
+	)
+	(junction
 		(at 177.8 62.23)
 		(diameter 0)
@@
 	)
 	(junction
+		(at 161.29 49.53)
+		(diameter 0)
+		(color 0 0 0 0)
+	)
+	(junction
 		(at 146.05 135.89)
 		(diameter 0)
@@
 	(wire
 		(pts
+			(xy 147.32 52.07) (xy 147.32 62.23)
+		)
+		(stroke
+			(width 0)
+			(type default)
+		)
+	)
+	(wire
+		(pts
 			(xy 284.48 130.81) (xy 289.56 130.81)
 		)
@@
 	(wire
 		(pts
+			(xy 147.32 49.53) (xy 161.29 49.53)
+		)
+		(stroke
+			(width 0)
+			(type default)
+		)
+	)
+	(wire
+		(pts
+			(xy 147.32 62.23) (xy 157.48 62.23)
+		)
+		(stroke
+			(width 0)
+			(type default)
+		)
+	)
+	(wire
+		(pts
 			(xy 143.51 135.89) (xy 146.05 135.89)
 		)
@@
 					(unit 1)
 				)
+			)
+		)
+	)
+	(symbol
+		(lib_id "Connector:Screw_Terminal_01x02")
+		(at 142.24 49.53 0)
+		(mirror y)
+		(unit 1)
+		(body_style 1)
+		(exclude_from_sim no)
+		(in_bom yes)
+		(on_board yes)
+		(in_pos_files yes)
+		(dnp no)
+		(fields_autoplaced yes)
+		(property "Reference" "J1602"
+			(at 142.24 43.18 0)
+			(show_name no)
+			(do_not_autoplace no)
+			(effects
+				(font
+					(size 1.27 1.27)
+				)
+			)
+		)
+		(property "Value" "Screw_Terminal_01x02"
+			(at 142.24 45.72 0)
+			(show_name no)
+			(do_not_autoplace no)
+			(effects
+				(font
+					(size 1.27 1.27)
+				)
+			)
+		)
+		(property "Footprint" ""
+			(at 142.24 49.53 0)
+			(hide yes)
+			(show_name no)
+			(do_not_autoplace no)
+			(effects
+				(font
+					(size 1.27 1.27)
+				)
+			)
+		)
+		(property "Datasheet" ""
+			(at 142.24 49.53 0)
+			(hide yes)
+			(show_name no)
+			(do_not_autoplace no)
+			(effects
+				(font
+					(size 1.27 1.27)
+				)
+			)
+		)
+		(property "Description" "Generic screw terminal, single row, 01x02, script generated (kicad-library-utils/schlib/autogen/connector/)"
+			(at 142.24 49.53 0)
+			(hide yes)
+			(show_name no)
+			(do_not_autoplace no)
+			(effects
+				(font
+					(size 1.27 1.27)
+				)
+			)
+		)
+		(pin "2"
+		)
+		(pin "1"
+		)
+		(instances
+			(project "TB04_S4_addr"
+				(path "/d176c79b-dced-4d01-bcec-7dfd676fcfc2"
+					(reference "J1602")
+					(unit 1)
+				)
