File: ver2/hardware/TB04addr8bit_copy/ALU.kicad_sch (KiCad schematic)
At the start: 8 parts, among them J801 Conn_02x05_Odd_Even, J802 Conn_02x05_Odd_Even, J803 Conn_02x05_Odd_Even, J804 Conn_02x05_Odd_Even, J805 Conn_02x05_Odd_Even, J806 Conn_02x05_Odd_Even, J807 Conn_02x05_Odd_Even, J808 Conn_02x05_Odd_Even

Commit message: ver2: ロータリースイッチSR1712F-0109のフットプリントを作成／SW502をrotarySW_01x09へ差し替え
- データシート(SLH-232)の埋め込み画像を読み、穴位置を実測して寸法を確定
  端子10-Ø0.9(2列×5・ピッチ2.5・列間18.3)、取付2-Ø2.0(間隔16.0・中点から1.1)
- KiCAD標準のSW_Rotary_1x9_MPは実物とピン番号が逆(pin10がコモン)だったため
  My_Lib:rotarySW_01x09(pin1=コモン)へ差し替え。実物・シンボル・FPが三者一致
- pcbnewのAPIでパッド12個の座標を全数検証
- マスターにfp-lib-tableを追加(footprints/Library.pretty)

Co-Authored-By: Claude Opus 5 <noreply@anthropic.com>
Parts:
- J801, J802, J803, J804, J805, J806, J807, J808: footprint (none) -> Connector_PinSocket_2.54mm:PinSocket_2x05_P2.54mm_Vertical
Changed lines of the file:
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@@
 		)
 		(instances
-			(project "TB04addr8bit"
+			(project "TB04addr8bit_copy"
 				(path "/d176c79b-dced-4d01-bcec-7dfd676fcfc2/8128481a-591d-4f1a-bdfd-fb80959a87d7"
 					(reference "#PWR0803")
@@
 			)
 		)
-		(property "Footprint" ""
+		(property "Footprint" "Connector_PinSocket_2.54mm:PinSocket_2x05_P2.54mm_Vertical"
 			(at 73.66 115.57 0)
 			(hide yes)
@@
 		)
 		(instances
-			(project "TB04addr8bit"
+			(project "TB04addr8bit_copy"
 				(path "/d176c79b-dced-4d01-bcec-7dfd676fcfc2/8128481a-591d-4f1a-bdfd-fb80959a87d7"
 					(reference "J806")
@@
 			)
 		)
-		(property "Footprint" ""
+		(property "Footprint" "Connector_PinSocket_2.54mm:PinSocket_2x05_P2.54mm_Vertical"
 			(at 137.16 40.64 0)
 			(hide yes)
@@
 		)
 		(instances
-			(project "TB04addr8bit"
+			(project "TB04addr8bit_copy"
 				(path "/d176c79b-dced-4d01-bcec-7dfd676fcfc2/8128481a-591d-4f1a-bdfd-fb80959a87d7"
 					(reference "J803")
@@
 		)
 		(instances
-			(project "TB04addr8bit"
+			(project "TB04addr8bit_copy"
 				(path "/d176c79b-dced-4d01-bcec-7dfd676fcfc2/8128481a-591d-4f1a-bdfd-fb80959a87d7"
 					(reference "#PWR0802")
@@
 			)
 		)
-		(property "Footprint" ""
+		(property "Footprint" "Connector_PinSocket_2.54mm:PinSocket_2x05_P2.54mm_Vertical"
 			(at 91.44 50.8 0)
 			(hide yes)
@@
 		)
 		(instances
-			(project "TB04addr8bit"
+			(project "TB04addr8bit_copy"
 				(path "/d176c79b-dced-4d01-bcec-7dfd676fcfc2/8128481a-591d-4f1a-bdfd-fb80959a87d7"
 					(reference "J802")
@@
 		)
 		(instances
-			(project "TB04addr8bit"
+			(project "TB04addr8bit_copy"
 				(path "/d176c79b-dced-4d01-bcec-7dfd676fcfc2/8128481a-591d-4f1a-bdfd-fb80959a87d7"
 					(reference "#PWR0805")
@@
 			)
 		)
-		(property "Footprint" ""
+		(property "Footprint" "Connector_PinSocket_2.54mm:PinSocket_2x05_P2.54mm_Vertical"
 			(at 157.48 50.8 0)
 			(hide yes)
@@
 		)
 		(instances
-			(project "TB04addr8bit"
+			(project "TB04addr8bit_copy"
 				(path "/d176c79b-dced-4d01-bcec-7dfd676fcfc2/8128481a-591d-4f1a-bdfd-fb80959a87d7"
 					(reference "J804")
@@
 			)
 		)
-		(property "Footprint" ""
+		(property "Footprint" "Connector_PinSocket_2.54mm:PinSocket_2x05_P2.54mm_Vertical"
 			(at 71.12 40.64 0)
 			(hide yes)
@@
 		)
 		(instances
-			(project "TB04addr8bit"
+			(project "TB04addr8bit_copy"
 				(path "/d176c79b-dced-4d01-bcec-7dfd676fcfc2/8128481a-591d-4f1a-bdfd-fb80959a87d7"
 					(reference "J801")
@@
 			)
 		)
-		(property "Footprint" ""
+		(property "Footprint" "Connector_PinSocket_2.54mm:PinSocket_2x05_P2.54mm_Vertical"
 			(at 93.98 124.46 0)
 			(hide yes)
@@
 		)
 		(instances
-			(project "TB04addr8bit"
+			(project "TB04addr8bit_copy"
 				(path "/d176c79b-dced-4d01-bcec-7dfd676fcfc2/8128481a-591d-4f1a-bdfd-fb80959a87d7"
 					(reference "J805")
@@
 		)
 		(instances
-			(project "TB04addr8bit"
+			(project "TB04addr8bit_copy"
 				(path "/d176c79b-dced-4d01-bcec-7dfd676fcfc2/8128481a-591d-4f1a-bdfd-fb80959a87d7"
 					(reference "#PWR0801")
@@
 		)
 		(instances
-			(project "TB04addr8bit"
+			(project "TB04addr8bit_copy"
 				(path "/d176c79b-dced-4d01-bcec-7dfd676fcfc2/8128481a-591d-4f1a-bdfd-fb80959a87d7"
 					(reference "#PWR0806")
@@
 			)
 		)
-		(property "Footprint" ""
+		(property "Footprint" "Connector_PinSocket_2.54mm:PinSocket_2x05_P2.54mm_Vertical"
 			(at 95.25 195.58 0)
 			(hide yes)
@@
 		)
 		(instances
-			(project "TB04addr8bit"
+			(project "TB04addr8bit_copy"
 				(path "/d176c79b-dced-4d01-bcec-7dfd676fcfc2/8128481a-591d-4f1a-bdfd-fb80959a87d7"
 					(reference "J807")
@@
 			)
 		)
-		(property "Footprint" ""
+		(property "Footprint" "Connector_PinSocket_2.54mm:PinSocket_2x05_P2.54mm_Vertical"
 			(at 72.39 179.07 0)
 			(hide yes)
@@
 		)
 		(instances
-			(project "TB04addr8bit"
+			(project "TB04addr8bit_copy"
 				(path "/d176c79b-dced-4d01-bcec-7dfd676fcfc2/8128481a-591d-4f1a-bdfd-fb80959a87d7"
 					(reference "J808")
@@
 		)
 		(instances
-			(project "TB04addr8bit"
+			(project "TB04addr8bit_copy"
 				(path "/d176c79b-dced-4d01-bcec-7dfd676fcfc2/8128481a-591d-4f1a-bdfd-fb80959a87d7"
 					(reference "#PWR0808")
@@
 		)
 		(instances
-			(project "TB04addr8bit"
+			(project "TB04addr8bit_copy"
 				(path "/d176c79b-dced-4d01-bcec-7dfd676fcfc2/8128481a-591d-4f1a-bdfd-fb80959a87d7"
 					(reference "#PWR0807")
@@
 		)
 		(instances
-			(project "TB04addr8bit"
+			(project "TB04addr8bit_copy"
 				(path "/d176c79b-dced-4d01-bcec-7dfd676fcfc2/8128481a-591d-4f1a-bdfd-fb80959a87d7"
 					(reference "#PWR0804")
