File: ver2/hardware/TB04addr8bit_copy/ram.kicad_sch (KiCad schematic)
At the start: 6 parts, among them U1101 6116, U1102 74HC244, U1103 74HC244

Commit message: ver2: ロータリースイッチSR1712F-0109のフットプリントを作成／SW502をrotarySW_01x09へ差し替え
- データシート(SLH-232)の埋め込み画像を読み、穴位置を実測して寸法を確定
  端子10-Ø0.9(2列×5・ピッチ2.5・列間18.3)、取付2-Ø2.0(間隔16.0・中点から1.1)
- KiCAD標準のSW_Rotary_1x9_MPは実物とピン番号が逆(pin10がコモン)だったため
  My_Lib:rotarySW_01x09(pin1=コモン)へ差し替え。実物・シンボル・FPが三者一致
- pcbnewのAPIでパッド12個の座標を全数検証
- マスターにfp-lib-tableを追加(footprints/Library.pretty)

Co-Authored-By: Claude Opus 5 <noreply@anthropic.com>
Parts:
- C1101, C1102, C1103: footprint (none) -> Capacitor_THT:C_Disc_D4.3mm_W1.9mm_P5.00mm
- U1101, U1103: footprint (none) -> Package_DIP:DIP-24_18.0mmx34.29mm_W15.24mm_Socket
- U1102: footprint (none) -> Package_DIP:DIP-20_W7.62mm_Socket
Changed lines of the file:
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@@
 		)
 		(instances
-			(project "TB04addr8bit"
+			(project "TB04addr8bit_copy"
 				(path "/d176c79b-dced-4d01-bcec-7dfd676fcfc2/d4d6bce3-987f-46b3-a9b7-788703d534f1"
 					(reference "#PWR01104")
@@
 			)
 		)
-		(property "Footprint" ""
+		(property "Footprint" "Capacitor_THT:C_Disc_D4.3mm_W1.9mm_P5.00mm"
 			(at 270.8148 30.48 0)
 			(hide yes)
@@
 		)
 		(instances
-			(project "TB04addr8bit"
+			(project "TB04addr8bit_copy"
 				(path "/d176c79b-dced-4d01-bcec-7dfd676fcfc2/d4d6bce3-987f-46b3-a9b7-788703d534f1"
 					(reference "C1103")
@@
 			)
 		)
-		(property "Footprint" ""
+		(property "Footprint" "Capacitor_THT:C_Disc_D4.3mm_W1.9mm_P5.00mm"
 			(at 88.9 29.5148 0)
 			(hide yes)
@@
 		)
 		(instances
-			(project "TB04addr8bit"
+			(project "TB04addr8bit_copy"
 				(path "/d176c79b-dced-4d01-bcec-7dfd676fcfc2/d4d6bce3-987f-46b3-a9b7-788703d534f1"
 					(reference "C1101")
@@
 		)
 		(instances
-			(project "TB04addr8bit"
+			(project "TB04addr8bit_copy"
 				(path "/d176c79b-dced-4d01-bcec-7dfd676fcfc2/d4d6bce3-987f-46b3-a9b7-788703d534f1"
 					(reference "#PWR01103")
@@
 		)
 		(instances
-			(project "TB04addr8bit"
+			(project "TB04addr8bit_copy"
 				(path "/d176c79b-dced-4d01-bcec-7dfd676fcfc2/d4d6bce3-987f-46b3-a9b7-788703d534f1"
 					(reference "#PWR01102")
@@
 			)
 		)
-		(property "Footprint" ""
+		(property "Footprint" "Package_DIP:DIP-24_18.0mmx34.29mm_W15.24mm_Socket"
 			(at 198.12 127 0)
 			(hide yes)
@@
 		)
 		(instances
-			(project "TB04addr8bit"
+			(project "TB04addr8bit_copy"
 				(path "/d176c79b-dced-4d01-bcec-7dfd676fcfc2/d4d6bce3-987f-46b3-a9b7-788703d534f1"
 					(reference "U1103")
@@
 			)
 		)
-		(property "Footprint" ""
+		(property "Footprint" "Package_DIP:DIP-24_18.0mmx34.29mm_W15.24mm_Socket"
 			(at 77.47 44.45 0)
 			(hide yes)
@@
 		)
 		(instances
-			(project "TB04addr8bit"
+			(project "TB04addr8bit_copy"
 				(path "/d176c79b-dced-4d01-bcec-7dfd676fcfc2/d4d6bce3-987f-46b3-a9b7-788703d534f1"
 					(reference "U1101")
@@
 		)
 		(instances
-			(project "TB04addr8bit"
+			(project "TB04addr8bit_copy"
 				(path "/d176c79b-dced-4d01-bcec-7dfd676fcfc2/d4d6bce3-987f-46b3-a9b7-788703d534f1"
 					(reference "#PWR01101")
@@
 			)
 		)
-		(property "Footprint" ""
+		(property "Footprint" "Capacitor_THT:C_Disc_D4.3mm_W1.9mm_P5.00mm"
 			(at 259.3848 30.48 0)
 			(hide yes)
@@
 		)
 		(instances
-			(project "TB04addr8bit"
+			(project "TB04addr8bit_copy"
 				(path "/d176c79b-dced-4d01-bcec-7dfd676fcfc2/d4d6bce3-987f-46b3-a9b7-788703d534f1"
 					(reference "C1102")
@@
 			)
 		)
-		(property "Footprint" ""
+		(property "Footprint" "Package_DIP:DIP-20_W7.62mm_Socket"
 			(at 191.77 55.88 0)
 			(hide yes)
@@
 		)
 		(instances
-			(project "TB04addr8bit"
+			(project "TB04addr8bit_copy"
 				(path "/d176c79b-dced-4d01-bcec-7dfd676fcfc2/d4d6bce3-987f-46b3-a9b7-788703d534f1"
 					(reference "U1102")
@@
 		)
 		(instances
-			(project "TB04addr8bit"
+			(project "TB04addr8bit_copy"
 				(path "/d176c79b-dced-4d01-bcec-7dfd676fcfc2/d4d6bce3-987f-46b3-a9b7-788703d534f1"
 					(reference "#PWR01105")

Commit message: ver2: PCBの粗配置を自動生成(回路図シートごとのブロック配置)
- 参照番号の百の位でグループ化し、各グループを矩形にまとめて配置
- グループ間の接続本数から順序を焼きなましで最適化(蛇行配置)
- 部品の重なり0・グループ矩形の重なり0を確認
- 基板内202個/はみ出し77個(3段目の下半分)。配線は未着手

Co-Authored-By: Claude Opus 5 <noreply@anthropic.com>
Parts:
- U1103: footprint Package_DIP:DIP-24_18.0mmx34.29mm_W15.24mm_Socket -> Package_DIP:DIP-20_W7.62mm_Socket
Changed lines of the file:
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@@
 			)
 		)
-		(property "Footprint" "Package_DIP:DIP-24_18.0mmx34.29mm_W15.24mm_Socket"
+		(property "Footprint" "Package_DIP:DIP-20_W7.62mm_Socket"
 			(at 198.12 127 0)
 			(hide yes)
