File: ver2/hardware/TB04addr8bit_copy/AddrDecord.kicad_sch (KiCad schematic)
At the start: 2 parts, among them U1301 74LS08

Commit message: ver2: ロータリースイッチSR1712F-0109のフットプリントを作成／SW502をrotarySW_01x09へ差し替え
- データシート(SLH-232)の埋め込み画像を読み、穴位置を実測して寸法を確定
  端子10-Ø0.9(2列×5・ピッチ2.5・列間18.3)、取付2-Ø2.0(間隔16.0・中点から1.1)
- KiCAD標準のSW_Rotary_1x9_MPは実物とピン番号が逆(pin10がコモン)だったため
  My_Lib:rotarySW_01x09(pin1=コモン)へ差し替え。実物・シンボル・FPが三者一致
- pcbnewのAPIでパッド12個の座標を全数検証
- マスターにfp-lib-tableを追加(footprints/Library.pretty)

Co-Authored-By: Claude Opus 5 <noreply@anthropic.com>
Parts:
- C1301: footprint (none) -> Capacitor_THT:C_Disc_D4.3mm_W1.9mm_P5.00mm
- U1301: footprint (none) -> Package_DIP:DIP-14_W7.62mm_Socket
Changed lines of the file:
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@@
 		)
 		(instances
-			(project "TB04addr8bit"
+			(project "TB04addr8bit_copy"
 				(path "/d176c79b-dced-4d01-bcec-7dfd676fcfc2/5966379b-e25d-4be9-810c-b95428770124"
 					(reference "#PWR01301")
@@
 			)
 		)
-		(property "Footprint" ""
+		(property "Footprint" "Capacitor_THT:C_Disc_D4.3mm_W1.9mm_P5.00mm"
 			(at 120.65 93.0148 0)
 			(hide yes)
@@
 		)
 		(instances
-			(project "TB04addr8bit"
+			(project "TB04addr8bit_copy"
 				(path "/d176c79b-dced-4d01-bcec-7dfd676fcfc2/5966379b-e25d-4be9-810c-b95428770124"
 					(reference "C1301")
@@
 		)
 		(instances
-			(project "TB04addr8bit"
+			(project "TB04addr8bit_copy"
 				(path "/d176c79b-dced-4d01-bcec-7dfd676fcfc2/5966379b-e25d-4be9-810c-b95428770124"
 					(reference "#PWR01302")
@@
 			)
 		)
-		(property "Footprint" ""
+		(property "Footprint" "Package_DIP:DIP-14_W7.62mm_Socket"
 			(at 67.31 62.23 0)
 			(hide yes)
@@
 		)
 		(instances
-			(project "TB04addr8bit"
+			(project "TB04addr8bit_copy"
 				(path "/d176c79b-dced-4d01-bcec-7dfd676fcfc2/5966379b-e25d-4be9-810c-b95428770124"
 					(reference "U1301")
@@
 			)
 		)
-		(property "Footprint" ""
+		(property "Footprint" "Package_DIP:DIP-14_W7.62mm_Socket"
 			(at 119.38 67.31 0)
 			(hide yes)
@@
 		)
 		(instances
-			(project "TB04addr8bit"
+			(project "TB04addr8bit_copy"
 				(path "/d176c79b-dced-4d01-bcec-7dfd676fcfc2/5966379b-e25d-4be9-810c-b95428770124"
 					(reference "U1301")
@@
 			)
 		)
-		(property "Footprint" ""
+		(property "Footprint" "Package_DIP:DIP-14_W7.62mm_Socket"
 			(at 92.71 59.69 0)
 			(hide yes)
@@
 		)
 		(instances
-			(project "TB04addr8bit"
+			(project "TB04addr8bit_copy"
 				(path "/d176c79b-dced-4d01-bcec-7dfd676fcfc2/5966379b-e25d-4be9-810c-b95428770124"
 					(reference "U1301")
@@
 			)
 		)
-		(property "Footprint" ""
+		(property "Footprint" "Package_DIP:DIP-14_W7.62mm_Socket"
 			(at 107.95 113.03 0)
 			(hide yes)
@@
 		)
 		(instances
-			(project "TB04addr8bit"
+			(project "TB04addr8bit_copy"
 				(path "/d176c79b-dced-4d01-bcec-7dfd676fcfc2/5966379b-e25d-4be9-810c-b95428770124"
 					(reference "U1301")
@@
 			)
 		)
-		(property "Footprint" ""
+		(property "Footprint" "Package_DIP:DIP-14_W7.62mm_Socket"
 			(at 67.31 40.64 0)
 			(hide yes)
@@
 		)
 		(instances
-			(project "TB04addr8bit"
+			(project "TB04addr8bit_copy"
 				(path "/d176c79b-dced-4d01-bcec-7dfd676fcfc2/5966379b-e25d-4be9-810c-b95428770124"
 					(reference "U1301")

Commit message: ver2: 分割元TB04addr8bit_copyの74LS表記もHCへ(Valueのみ56件)
3分割と同じスクリプトを適用。置換56件は3分割の合計と一致。
副産物として、3分割の合計と_copyの品種別パッケージ数が全数一致
(253x12/161Nx11/244x10/273x6/157x4/377x4ほか計61)することを確認
= ICの取りこぼし・重複がないことの独立した裏づけ。

検証: 残存する74LSのValue 0件、変更行はValueの56行のみ
凍結マスターTB04addr8bitは08-23の状態で古いため対象外

Co-Authored-By: Claude Opus 5 <noreply@anthropic.com>
Parts:
- U1301: value 74LS08 -> 74HC08
Changed lines of the file:
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@@
 			)
 		)
-		(property "Value" "74LS08"
+		(property "Value" "74HC08"
 			(at 67.3017 55.88 0)
 			(show_name no)
@@
 			)
 		)
-		(property "Value" "74LS08"
+		(property "Value" "74HC08"
 			(at 119.3717 60.96 0)
 			(show_name no)
@@
 			)
 		)
-		(property "Value" "74LS08"
+		(property "Value" "74HC08"
 			(at 92.7017 53.34 0)
 			(show_name no)
@@
 			)
 		)
-		(property "Value" "74LS08"
+		(property "Value" "74HC08"
 			(at 114.3 114.2999 0)
 			(show_name no)
@@
 			)
 		)
-		(property "Value" "74LS08"
+		(property "Value" "74HC08"
 			(at 67.3017 34.29 0)
 			(show_name no)
