File: ver2/hardware/TB04addr8bit_copy/ROM_ALU.kicad_sch (KiCad schematic)
At the start: 31 parts, among them IC601 74HC161N, J601 Conn_02x05_Odd_Even, SW601 SW_Coded_SH-7050, U601 74LS273, U602 74HC273, U603 28C256, U604 28C256, U605 74HC74, U606 74HC273, U607 74HC238

Commit message: ver2: ロータリースイッチSR1712F-0109のフットプリントを作成／SW502をrotarySW_01x09へ差し替え
- データシート(SLH-232)の埋め込み画像を読み、穴位置を実測して寸法を確定
  端子10-Ø0.9(2列×5・ピッチ2.5・列間18.3)、取付2-Ø2.0(間隔16.0・中点から1.1)
- KiCAD標準のSW_Rotary_1x9_MPは実物とピン番号が逆(pin10がコモン)だったため
  My_Lib:rotarySW_01x09(pin1=コモン)へ差し替え。実物・シンボル・FPが三者一致
- pcbnewのAPIでパッド12個の座標を全数検証
- マスターにfp-lib-tableを追加(footprints/Library.pretty)

Co-Authored-By: Claude Opus 5 <noreply@anthropic.com>
Parts:
- J601: footprint (none) -> Connector_PinSocket_2.54mm:PinSocket_2x05_P2.54mm_Vertical
- R603, R604, R605, R606: footprint (none) -> Resistor_THT:R_Axial_DIN0207_L6.3mm_D2.5mm_P10.16mm_Horizontal
- SW601: footprint (none) -> Library:dip_rotary_sw

Commit message: ver2: 分割元TB04addr8bit_copyの74LS表記もHCへ(Valueのみ56件)
3分割と同じスクリプトを適用。置換56件は3分割の合計と一致。
副産物として、3分割の合計と_copyの品種別パッケージ数が全数一致
(253x12/161Nx11/244x10/273x6/157x4/377x4ほか計61)することを確認
= ICの取りこぼし・重複がないことの独立した裏づけ。

検証: 残存する74LSのValue 0件、変更行はValueの56行のみ
凍結マスターTB04addr8bitは08-23の状態で古いため対象外

Co-Authored-By: Claude Opus 5 <noreply@anthropic.com>
Parts:
- U601: value 74LS273 -> 74HC273
Changed lines of the file:
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@@
 			)
 		)
-		(property "Value" "74LS273"
+		(property "Value" "74HC273"
 			(at 366.6333 38.1 0)
 			(show_name no)
