File: ver2/hardware/TB04addr8bit_copy/RS01.kicad_sch (KiCad schematic)
At the start: 20 parts, among them IC301 74HC161N, IC302 74HC161N, IC303 74HC161N, IC304 74HC161N, J301 Conn_02x05_Odd_Even, J302 Conn_02x05_Odd_Even, J303 Conn_02x05_Odd_Even, J304 Conn_02x05_Odd_Even, U301 74LS253, U302 74LS253, U303 74LS253, U304 74LS253

Commit message: ver2: ロータリースイッチSR1712F-0109のフットプリントを作成／SW502をrotarySW_01x09へ差し替え
- データシート(SLH-232)の埋め込み画像を読み、穴位置を実測して寸法を確定
  端子10-Ø0.9(2列×5・ピッチ2.5・列間18.3)、取付2-Ø2.0(間隔16.0・中点から1.1)
- KiCAD標準のSW_Rotary_1x9_MPは実物とピン番号が逆(pin10がコモン)だったため
  My_Lib:rotarySW_01x09(pin1=コモン)へ差し替え。実物・シンボル・FPが三者一致
- pcbnewのAPIでパッド12個の座標を全数検証
- マスターにfp-lib-tableを追加(footprints/Library.pretty)

Co-Authored-By: Claude Opus 5 <noreply@anthropic.com>
Parts:
- J301, J302, J303, J304: footprint (none) -> Connector_PinSocket_2.54mm:PinSocket_2x05_P2.54mm_Vertical
Changed lines of the file:
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@@
 		)
 		(instances
-			(project "TB04addr8bit"
+			(project "TB04addr8bit_copy"
 				(path "/d176c79b-dced-4d01-bcec-7dfd676fcfc2/87662b34-7613-4342-918c-9ae2f7d081f7"
 					(reference "#PWR0316")
@@
 		)
 		(instances
-			(project "TB04addr8bit"
+			(project "TB04addr8bit_copy"
 				(path "/d176c79b-dced-4d01-bcec-7dfd676fcfc2/87662b34-7613-4342-918c-9ae2f7d081f7"
 					(reference "#PWR0317")
@@
 		)
 		(instances
-			(project "TB04addr8bit"
+			(project "TB04addr8bit_copy"
 				(path "/d176c79b-dced-4d01-bcec-7dfd676fcfc2/87662b34-7613-4342-918c-9ae2f7d081f7"
 					(reference "#PWR0305")
@@
 		)
 		(instances
-			(project "TB04addr8bit"
+			(project "TB04addr8bit_copy"
 				(path "/d176c79b-dced-4d01-bcec-7dfd676fcfc2/87662b34-7613-4342-918c-9ae2f7d081f7"
 					(reference "#PWR0307")
@@
 		)
 		(instances
-			(project "TB04addr8bit"
+			(project "TB04addr8bit_copy"
 				(path "/d176c79b-dced-4d01-bcec-7dfd676fcfc2/87662b34-7613-4342-918c-9ae2f7d081f7"
 					(reference "IC302")
@@
 		)
 		(instances
-			(project "TB04addr8bit"
+			(project "TB04addr8bit_copy"
 				(path "/d176c79b-dced-4d01-bcec-7dfd676fcfc2/87662b34-7613-4342-918c-9ae2f7d081f7"
 					(reference "C302")
@@
 			)
 		)
-		(property "Footprint" ""
+		(property "Footprint" "Connector_PinSocket_2.54mm:PinSocket_2x05_P2.54mm_Vertical"
 			(at 215.9 62.23 0)
 			(hide yes)
@@
 		)
 		(instances
-			(project "TB04addr8bit"
+			(project "TB04addr8bit_copy"
 				(path "/d176c79b-dced-4d01-bcec-7dfd676fcfc2/87662b34-7613-4342-918c-9ae2f7d081f7"
 					(reference "J302")
@@
 		)
 		(instances
-			(project "TB04addr8bit"
+			(project "TB04addr8bit_copy"
 				(path "/d176c79b-dced-4d01-bcec-7dfd676fcfc2/87662b34-7613-4342-918c-9ae2f7d081f7"
 					(reference "#PWR0318")
@@
 		)
 		(instances
-			(project "TB04addr8bit"
+			(project "TB04addr8bit_copy"
 				(path "/d176c79b-dced-4d01-bcec-7dfd676fcfc2/87662b34-7613-4342-918c-9ae2f7d081f7"
 					(reference "C305")
@@
 		)
 		(instances
-			(project "TB04addr8bit"
+			(project "TB04addr8bit_copy"
 				(path "/d176c79b-dced-4d01-bcec-7dfd676fcfc2/87662b34-7613-4342-918c-9ae2f7d081f7"
 					(reference "C306")
@@
 		)
 		(instances
-			(project "TB04addr8bit"
+			(project "TB04addr8bit_copy"
 				(path "/d176c79b-dced-4d01-bcec-7dfd676fcfc2/87662b34-7613-4342-918c-9ae2f7d081f7"
 					(reference "#PWR0320")
@@
 		)
 		(instances
-			(project "TB04addr8bit"
+			(project "TB04addr8bit_copy"
 				(path "/d176c79b-dced-4d01-bcec-7dfd676fcfc2/87662b34-7613-4342-918c-9ae2f7d081f7"
 					(reference "#PWR0308")
@@
 		)
 		(instances
-			(project "TB04addr8bit"
+			(project "TB04addr8bit_copy"
 				(path "/d176c79b-dced-4d01-bcec-7dfd676fcfc2/87662b34-7613-4342-918c-9ae2f7d081f7"
 					(reference "U301")
@@
 		)
 		(instances
-			(project "TB04addr8bit"
+			(project "TB04addr8bit_copy"
 				(path "/d176c79b-dced-4d01-bcec-7dfd676fcfc2/87662b34-7613-4342-918c-9ae2f7d081f7"
 					(reference "C304")
@@
 		)
 		(instances
-			(project "TB04addr8bit"
+			(project "TB04addr8bit_copy"
 				(path "/d176c79b-dced-4d01-bcec-7dfd676fcfc2/87662b34-7613-4342-918c-9ae2f7d081f7"
 					(reference "#PWR0311")
@@
 		)
 		(instances
-			(project "TB04addr8bit"
+			(project "TB04addr8bit_copy"
 				(path "/d176c79b-dced-4d01-bcec-7dfd676fcfc2/87662b34-7613-4342-918c-9ae2f7d081f7"
 					(reference "C307")
@@
 			)
 		)
-		(property "Footprint" ""
+		(property "Footprint" "Connector_PinSocket_2.54mm:PinSocket_2x05_P2.54mm_Vertical"
 			(at 157.48 158.75 0)
 			(hide yes)
@@
 		)
 		(instances
-			(project "TB04addr8bit"
+			(project "TB04addr8bit_copy"
 				(path "/d176c79b-dced-4d01-bcec-7dfd676fcfc2/87662b34-7613-4342-918c-9ae2f7d081f7"
 					(reference "J304")
@@
 		)
 		(instances
-			(project "TB04addr8bit"
+			(project "TB04addr8bit_copy"
 				(path "/d176c79b-dced-4d01-bcec-7dfd676fcfc2/87662b34-7613-4342-918c-9ae2f7d081f7"
 					(reference "#PWR0302")
@@
 		)
 		(instances
-			(project "TB04addr8bit"
+			(project "TB04addr8bit_copy"
 				(path "/d176c79b-dced-4d01-bcec-7dfd676fcfc2/87662b34-7613-4342-918c-9ae2f7d081f7"
 					(reference "#PWR0306")
@@
 		)
 		(instances
-			(project "TB04addr8bit"
+			(project "TB04addr8bit_copy"
 				(path "/d176c79b-dced-4d01-bcec-7dfd676fcfc2/87662b34-7613-4342-918c-9ae2f7d081f7"
 					(reference "#PWR0309")
@@
 		)
 		(instances
-			(project "TB04addr8bit"
+			(project "TB04addr8bit_copy"
 				(path "/d176c79b-dced-4d01-bcec-7dfd676fcfc2/87662b34-7613-4342-918c-9ae2f7d081f7"
 					(reference "IC301")
@@
 		)
 		(instances
-			(project "TB04addr8bit"
+			(project "TB04addr8bit_copy"
 				(path "/d176c79b-dced-4d01-bcec-7dfd676fcfc2/87662b34-7613-4342-918c-9ae2f7d081f7"
 					(reference "#PWR0315")
@@
 		)
 		(instances
-			(project "TB04addr8bit"
+			(project "TB04addr8bit_copy"
 				(path "/d176c79b-dced-4d01-bcec-7dfd676fcfc2/87662b34-7613-4342-918c-9ae2f7d081f7"
 					(reference "#PWR0310")
@@
 		)
 		(instances
-			(project "TB04addr8bit"
+			(project "TB04addr8bit_copy"
 				(path "/d176c79b-dced-4d01-bcec-7dfd676fcfc2/87662b34-7613-4342-918c-9ae2f7d081f7"
 					(reference "#PWR0312")
@@
 		)
 		(instances
-			(project "TB04addr8bit"
+			(project "TB04addr8bit_copy"
 				(path "/d176c79b-dced-4d01-bcec-7dfd676fcfc2/87662b34-7613-4342-918c-9ae2f7d081f7"
 					(reference "C303")
@@
 			)
 		)
-		(property "Footprint" ""
+		(property "Footprint" "Connector_PinSocket_2.54mm:PinSocket_2x05_P2.54mm_Vertical"
 			(at 166.37 67.31 0)
 			(hide yes)
@@
 		)
 		(instances
-			(project "TB04addr8bit"
+			(project "TB04addr8bit_copy"
 				(path "/d176c79b-dced-4d01-bcec-7dfd676fcfc2/87662b34-7613-4342-918c-9ae2f7d081f7"
 					(reference "J301")
@@
 		)
 		(instances
-			(project "TB04addr8bit"
+			(project "TB04addr8bit_copy"
 				(path "/d176c79b-dced-4d01-bcec-7dfd676fcfc2/87662b34-7613-4342-918c-9ae2f7d081f7"
 					(reference "#PWR0303")
@@
 		)
 		(instances
-			(project "TB04addr8bit"
+			(project "TB04addr8bit_copy"
 				(path "/d176c79b-dced-4d01-bcec-7dfd676fcfc2/87662b34-7613-4342-918c-9ae2f7d081f7"
 					(reference "#PWR0313")
@@
 		)
 		(instances
-			(project "TB04addr8bit"
+			(project "TB04addr8bit_copy"
 				(path "/d176c79b-dced-4d01-bcec-7dfd676fcfc2/87662b34-7613-4342-918c-9ae2f7d081f7"
 					(reference "U303")
@@
 		)
 		(instances
-			(project "TB04addr8bit"
+			(project "TB04addr8bit_copy"
 				(path "/d176c79b-dced-4d01-bcec-7dfd676fcfc2/87662b34-7613-4342-918c-9ae2f7d081f7"
 					(reference "U302")
@@
 		)
 		(instances
-			(project "TB04addr8bit"
+			(project "TB04addr8bit_copy"
 				(path "/d176c79b-dced-4d01-bcec-7dfd676fcfc2/87662b34-7613-4342-918c-9ae2f7d081f7"
 					(reference "U304")
@@
 		)
 		(instances
-			(project "TB04addr8bit"
+			(project "TB04addr8bit_copy"
 				(path "/d176c79b-dced-4d01-bcec-7dfd676fcfc2/87662b34-7613-4342-918c-9ae2f7d081f7"
 					(reference "IC304")
@@
 		)
 		(instances
-			(project "TB04addr8bit"
+			(project "TB04addr8bit_copy"
 				(path "/d176c79b-dced-4d01-bcec-7dfd676fcfc2/87662b34-7613-4342-918c-9ae2f7d081f7"
 					(reference "#PWR0319")
@@
 			)
 		)
-		(property "Footprint" ""
+		(property "Footprint" "Connector_PinSocket_2.54mm:PinSocket_2x05_P2.54mm_Vertical"
 			(at 176.53 105.41 0)
 			(hide yes)
@@
 		)
 		(instances
-			(project "TB04addr8bit"
+			(project "TB04addr8bit_copy"
 				(path "/d176c79b-dced-4d01-bcec-7dfd676fcfc2/87662b34-7613-4342-918c-9ae2f7d081f7"
 					(reference "J303")
@@
 		)
 		(instances
-			(project "TB04addr8bit"
+			(project "TB04addr8bit_copy"
 				(path "/d176c79b-dced-4d01-bcec-7dfd676fcfc2/87662b34-7613-4342-918c-9ae2f7d081f7"
 					(reference "#PWR0301")
@@
 		)
 		(instances
-			(project "TB04addr8bit"
+			(project "TB04addr8bit_copy"
 				(path "/d176c79b-dced-4d01-bcec-7dfd676fcfc2/87662b34-7613-4342-918c-9ae2f7d081f7"
 					(reference "C301")
@@
 		)
 		(instances
-			(project "TB04addr8bit"
+			(project "TB04addr8bit_copy"
 				(path "/d176c79b-dced-4d01-bcec-7dfd676fcfc2/87662b34-7613-4342-918c-9ae2f7d081f7"
 					(reference "IC303")
@@
 		)
 		(instances
-			(project "TB04addr8bit"
+			(project "TB04addr8bit_copy"
 				(path "/d176c79b-dced-4d01-bcec-7dfd676fcfc2/87662b34-7613-4342-918c-9ae2f7d081f7"
 					(reference "#PWR0314")
@@
 		)
 		(instances
-			(project "TB04addr8bit"
+			(project "TB04addr8bit_copy"
 				(path "/d176c79b-dced-4d01-bcec-7dfd676fcfc2/87662b34-7613-4342-918c-9ae2f7d081f7"
 					(reference "#PWR0304")
@@
 		)
 		(instances
-			(project "TB04addr8bit"
+			(project "TB04addr8bit_copy"
 				(path "/d176c79b-dced-4d01-bcec-7dfd676fcfc2/87662b34-7613-4342-918c-9ae2f7d081f7"
 					(reference "C308")

Commit message: ver2: レジスタLED32個を追加し、それを織り込んでPCBを再配置
- 回路図にレジスタ表示LED(D2xx/D3xx)とSIP抵抗を追加(部品279→307)
- 密度は61.3%→62.4%でほぼ変わらず
- RS00/RS01を下端の帯の上に固定し、ブロック内でLEDを手前側へ
- 6xx/7xx/15xxを横長にして上部に収め、基板内14/16グループに改善
- 部品の重なり0・基板内281個/はみ出し26個

Co-Authored-By: Claude Opus 5 <noreply@anthropic.com>
Parts:
- removed J301, J302, J303, J304: Conn_02x05_Odd_Even, Connector_PinSocket_2.54mm:PinSocket_2x05_P2.54mm_Vertical, symbol Connector_Generic:Conn_02x05_Odd_Even
- added D301, D302, D303, D304, D305, D306, D307, D308, D309, D310, D311, D312, D313, D314, D315, D316: LED, LED_THT:LED_D3.0mm_Clear, symbol Device:LED
- added RN301, RN302: 4.7K, Resistor_THT:R_Array_SIP9, symbol Device:R_Network08
Connections:
- net GND: now also RN301.1 (common), RN302.1 (common)
- net I0a0: now also D316.2 (A)
- net I0a1: now also D308.2 (A)
- net I0a2: now also D315.2 (A)
- net I0a3: now also D307.2 (A)
- net I0b0: now also D314.2 (A)
- net I0b1: now also D306.2 (A)
- net I0b2: now also D313.2 (A)
- net I0b3: now also D305.2 (A)
- net I1a0: now also D312.2 (A)
- net I1a1: now also D304.2 (A)
- net I1a2: now also D311.2 (A)
- net I1a3: now also D303.2 (A)
- net I1b0: now also D310.2 (A)
- net I1b1: now also D302.2 (A)
- net I1b2: now also D309.2 (A)
- net I1b3: now also D301.2 (A)
- new net: D307.1 (K), RN301.5 (R4)
- new net: D306.1 (K), RN302.4 (R3)
- new net: D303.1 (K), RN301.3 (R2)
- new net: D311.1 (K), RN301.7 (R6)
- new net: D315.1 (K), RN301.9 (R8)
- new net: D301.1 (K), RN301.2 (R1)
- new net: D302.1 (K), RN302.2 (R1)
- new net: D316.1 (K), RN302.9 (R8)
- new net: D305.1 (K), RN301.4 (R3)
- new net: D309.1 (K), RN301.6 (R5)
- new net: D313.1 (K), RN301.8 (R7)
- new net: D308.1 (K), RN302.5 (R4)
- new net: D314.1 (K), RN302.8 (R7)
- new net: D304.1 (K), RN302.3 (R2)
- new net: D310.1 (K), RN302.6 (R5)
- new net: D312.1 (K), RN302.7 (R6)
- no-connect marks 16 -> 4

Commit message: ver2: 分割元TB04addr8bit_copyの74LS表記もHCへ(Valueのみ56件)
3分割と同じスクリプトを適用。置換56件は3分割の合計と一致。
副産物として、3分割の合計と_copyの品種別パッケージ数が全数一致
(253x12/161Nx11/244x10/273x6/157x4/377x4ほか計61)することを確認
= ICの取りこぼし・重複がないことの独立した裏づけ。

検証: 残存する74LSのValue 0件、変更行はValueの56行のみ
凍結マスターTB04addr8bitは08-23の状態で古いため対象外

Co-Authored-By: Claude Opus 5 <noreply@anthropic.com>
Parts:
- U301, U302, U303, U304: value 74LS253 -> 74HC253
Changed lines of the file:
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@@
 			)
 		)
-		(property "Value" "74LS253"
+		(property "Value" "74HC253"
 			(at 332.3433 24.13 0)
 			(show_name no)
@@
 			)
 		)
-		(property "Value" "74LS253"
+		(property "Value" "74HC253"
 			(at 267.5733 147.32 0)
 			(show_name no)
@@
 			)
 		)
-		(property "Value" "74LS253"
+		(property "Value" "74HC253"
 			(at 332.3433 101.6 0)
 			(show_name no)
@@
 			)
 		)
-		(property "Value" "74LS253"
+		(property "Value" "74HC253"
 			(at 299.3233 219.71 0)
 			(show_name no)
