File: ver2/hardware/TB04addr8bit_copy/TB04addr8bit_copy.kicad_sch (KiCad schematic)
At the start: 12 parts, among them J101 USB_C_Receptacle_PowerOnly_6P, SW101 SW_SPDT, U101 74LS157, U102 74HC138

Commit message: ver2: ロータリースイッチSR1712F-0109のフットプリントを作成／SW502をrotarySW_01x09へ差し替え
- データシート(SLH-232)の埋め込み画像を読み、穴位置を実測して寸法を確定
  端子10-Ø0.9(2列×5・ピッチ2.5・列間18.3)、取付2-Ø2.0(間隔16.0・中点から1.1)
- KiCAD標準のSW_Rotary_1x9_MPは実物とピン番号が逆(pin10がコモン)だったため
  My_Lib:rotarySW_01x09(pin1=コモン)へ差し替え。実物・シンボル・FPが三者一致
- pcbnewのAPIでパッド12個の座標を全数検証
- マスターにfp-lib-tableを追加(footprints/Library.pretty)

Co-Authored-By: Claude Opus 5 <noreply@anthropic.com>
Parts:
- U101: footprint (none) -> Package_DIP:DIP-16_W7.62mm_Socket
Changed lines of the file:
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@@
 				)
 			)
-			(project "TB04addr8bit"
+			(project "TB04addr8bit_copy"
 				(path "/d176c79b-dced-4d01-bcec-7dfd676fcfc2"
 					(reference "R102")
@@
 				)
 			)
-			(project "TB04addr8bit"
+			(project "TB04addr8bit_copy"
 				(path "/d176c79b-dced-4d01-bcec-7dfd676fcfc2"
 					(reference "#PWR0103")
@@
 				)
 			)
-			(project "TB04addr8bit"
+			(project "TB04addr8bit_copy"
 				(path "/d176c79b-dced-4d01-bcec-7dfd676fcfc2"
 					(reference "C104")
@@
 				)
 			)
-			(project "TB04addr8bit"
+			(project "TB04addr8bit_copy"
 				(path "/d176c79b-dced-4d01-bcec-7dfd676fcfc2"
 					(reference "#FLG0101")
@@
 				)
 			)
-			(project "TB04addr8bit"
+			(project "TB04addr8bit_copy"
 				(path "/d176c79b-dced-4d01-bcec-7dfd676fcfc2"
 					(reference "#FLG0102")
@@
 				)
 			)
-			(project "TB04addr8bit"
+			(project "TB04addr8bit_copy"
 				(path "/d176c79b-dced-4d01-bcec-7dfd676fcfc2"
 					(reference "#PWR0102")
@@
 				)
 			)
-			(project "TB04addr8bit"
+			(project "TB04addr8bit_copy"
 				(path "/d176c79b-dced-4d01-bcec-7dfd676fcfc2"
 					(reference "C103")
@@
 				)
 			)
-			(project "TB04addr8bit"
+			(project "TB04addr8bit_copy"
 				(path "/d176c79b-dced-4d01-bcec-7dfd676fcfc2"
 					(reference "R103")
@@
 		)
 		(instances
-			(project "TB04addr8bit"
+			(project "TB04addr8bit_copy"
 				(path "/d176c79b-dced-4d01-bcec-7dfd676fcfc2"
 					(reference "#PWR0107")
@@
 				)
 			)
-			(project "TB04addr8bit"
+			(project "TB04addr8bit_copy"
 				(path "/d176c79b-dced-4d01-bcec-7dfd676fcfc2"
 					(reference "#PWR0104")
@@
 				)
 			)
-			(project "TB04addr8bit"
+			(project "TB04addr8bit_copy"
 				(path "/d176c79b-dced-4d01-bcec-7dfd676fcfc2"
 					(reference "#PWR0105")
@@
 				)
 			)
-			(project "TB04addr8bit"
+			(project "TB04addr8bit_copy"
 				(path "/d176c79b-dced-4d01-bcec-7dfd676fcfc2"
 					(reference "J101")
@@
 		)
 		(instances
-			(project "TB04addr8bit"
+			(project "TB04addr8bit_copy"
 				(path "/d176c79b-dced-4d01-bcec-7dfd676fcfc2"
 					(reference "#PWR0101")
@@
 				)
 			)
-			(project "TB04addr8bit"
+			(project "TB04addr8bit_copy"
 				(path "/d176c79b-dced-4d01-bcec-7dfd676fcfc2"
 					(reference "R101")
@@
 				)
 			)
-			(project "TB04addr8bit"
+			(project "TB04addr8bit_copy"
 				(path "/d176c79b-dced-4d01-bcec-7dfd676fcfc2"
 					(reference "D101")
@@
 				)
 			)
-			(project "TB04addr8bit"
+			(project "TB04addr8bit_copy"
 				(path "/d176c79b-dced-4d01-bcec-7dfd676fcfc2"
 					(reference "#PWR0108")
@@
 				)
 			)
-			(project "TB04addr8bit"
+			(project "TB04addr8bit_copy"
 				(path "/d176c79b-dced-4d01-bcec-7dfd676fcfc2"
 					(reference "C102")
@@
 			)
 		)
-		(property "Footprint" ""
+		(property "Footprint" "Package_DIP:DIP-16_W7.62mm_Socket"
 			(at 171.45 146.05 0)
 			(hide yes)
@@
 		)
 		(instances
-			(project "TB04addr8bit"
+			(project "TB04addr8bit_copy"
 				(path "/d176c79b-dced-4d01-bcec-7dfd676fcfc2"
 					(reference "U101")
@@
 				)
 			)
-			(project "TB04addr8bit"
+			(project "TB04addr8bit_copy"
 				(path "/d176c79b-dced-4d01-bcec-7dfd676fcfc2"
 					(reference "#PWR0106")
@@
 				)
 			)
-			(project "TB04addr8bit"
+			(project "TB04addr8bit_copy"
 				(path "/d176c79b-dced-4d01-bcec-7dfd676fcfc2"
 					(reference "SW101")
@@
 		)
 		(instances
-			(project "TB04addr8bit"
+			(project "TB04addr8bit_copy"
 				(path "/d176c79b-dced-4d01-bcec-7dfd676fcfc2"
 					(reference "C101")
@@
 				)
 			)
-			(project "TB04addr8bit"
+			(project "TB04addr8bit_copy"
 				(path "/d176c79b-dced-4d01-bcec-7dfd676fcfc2"
 					(reference "U102")
@@
 				)
 			)
-			(project "TB04addr8bit"
+			(project "TB04addr8bit_copy"
 				(path "/d176c79b-dced-4d01-bcec-7dfd676fcfc2"
 					(page "6")
@@
 		)
 		(instances
-			(project "TB04addr8bit"
+			(project "TB04addr8bit_copy"
 				(path "/d176c79b-dced-4d01-bcec-7dfd676fcfc2"
 					(page "9")
@@
 		)
 		(instances
-			(project "TB04addr8bit"
+			(project "TB04addr8bit_copy"
 				(path "/d176c79b-dced-4d01-bcec-7dfd676fcfc2"
 					(page "12")
@@
 		)
 		(instances
-			(project "TB04addr8bit"
+			(project "TB04addr8bit_copy"
 				(path "/d176c79b-dced-4d01-bcec-7dfd676fcfc2"
 					(page "13")
@@
 		)
 		(instances
-			(project "TB04addr8bit"
+			(project "TB04addr8bit_copy"
 				(path "/d176c79b-dced-4d01-bcec-7dfd676fcfc2"
 					(page "15")
@@
 				)
 			)
-			(project "TB04addr8bit"
+			(project "TB04addr8bit_copy"
 				(path "/d176c79b-dced-4d01-bcec-7dfd676fcfc2"
 					(page "4")
@@
 				)
 			)
-			(project "TB04addr8bit"
+			(project "TB04addr8bit_copy"
 				(path "/d176c79b-dced-4d01-bcec-7dfd676fcfc2"
 					(page "8")
@@
 		)
 		(instances
-			(project "TB04addr8bit"
+			(project "TB04addr8bit_copy"
 				(path "/d176c79b-dced-4d01-bcec-7dfd676fcfc2"
 					(page "3")
@@
 				)
 			)
-			(project "TB04addr8bit"
+			(project "TB04addr8bit_copy"
 				(path "/d176c79b-dced-4d01-bcec-7dfd676fcfc2"
 					(page "5")
@@
 				)
 			)
-			(project "TB04addr8bit"
+			(project "TB04addr8bit_copy"
 				(path "/d176c79b-dced-4d01-bcec-7dfd676fcfc2"
 					(page "2")
@@
 		)
 		(instances
-			(project "TB04addr8bit"
+			(project "TB04addr8bit_copy"
 				(path "/d176c79b-dced-4d01-bcec-7dfd676fcfc2"
 					(page "10")
@@
 		)
 		(instances
-			(project "TB04addr8bit"
+			(project "TB04addr8bit_copy"
 				(path "/d176c79b-dced-4d01-bcec-7dfd676fcfc2"
 					(page "11")
@@
 		)
 		(instances
-			(project "TB04addr8bit"
+			(project "TB04addr8bit_copy"
 				(path "/d176c79b-dced-4d01-bcec-7dfd676fcfc2"
 					(page "14")
@@
 		)
 		(instances
-			(project "TB04addr8bit"
+			(project "TB04addr8bit_copy"
 				(path "/d176c79b-dced-4d01-bcec-7dfd676fcfc2"
 					(page "7")

Commit message: ver2: 分割元TB04addr8bit_copyの74LS表記もHCへ(Valueのみ56件)
3分割と同じスクリプトを適用。置換56件は3分割の合計と一致。
副産物として、3分割の合計と_copyの品種別パッケージ数が全数一致
(253x12/161Nx11/244x10/273x6/157x4/377x4ほか計61)することを確認
= ICの取りこぼし・重複がないことの独立した裏づけ。

検証: 残存する74LSのValue 0件、変更行はValueの56行のみ
凍結マスターTB04addr8bitは08-23の状態で古いため対象外

Co-Authored-By: Claude Opus 5 <noreply@anthropic.com>
Parts:
- U101: value 74LS157 -> 74HC157
Changed lines of the file:
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@@
 			)
 		)
-		(property "Value" "74LS157"
+		(property "Value" "74HC157"
 			(at 173.5933 125.73 0)
 			(show_name no)
