File: ver2/hardware/TB04addr8bit_copy/outPut.kicad_sch (KiCad schematic)
At the start: 32 parts, among them J901 Conn_02x05_Odd_Even, J902 Conn_02x05_Odd_Even, J903 Conn_02x05_Odd_Even, J904 Conn_02x05_Odd_Even, U901 74LS377, U902 74LS377, U903 74LS377, U905 74LS377

Commit message: ver2: ロータリースイッチSR1712F-0109のフットプリントを作成／SW502をrotarySW_01x09へ差し替え
- データシート(SLH-232)の埋め込み画像を読み、穴位置を実測して寸法を確定
  端子10-Ø0.9(2列×5・ピッチ2.5・列間18.3)、取付2-Ø2.0(間隔16.0・中点から1.1)
- KiCAD標準のSW_Rotary_1x9_MPは実物とピン番号が逆(pin10がコモン)だったため
  My_Lib:rotarySW_01x09(pin1=コモン)へ差し替え。実物・シンボル・FPが三者一致
- pcbnewのAPIでパッド12個の座標を全数検証
- マスターにfp-lib-tableを追加(footprints/Library.pretty)

Co-Authored-By: Claude Opus 5 <noreply@anthropic.com>
Parts:
- C901, C902, C903, C904: footprint (none) -> Capacitor_THT:C_Disc_D4.3mm_W1.9mm_P5.00mm
- J901, J902, J903, J904: footprint (none) -> Connector_PinSocket_2.54mm:PinSocket_2x05_P2.54mm_Vertical
- U901, U902, U903, U905: footprint (none) -> Package_DIP:DIP-20_W7.62mm_Socket

Commit message: ver2: 分割元TB04addr8bit_copyの74LS表記もHCへ(Valueのみ56件)
3分割と同じスクリプトを適用。置換56件は3分割の合計と一致。
副産物として、3分割の合計と_copyの品種別パッケージ数が全数一致
(253x12/161Nx11/244x10/273x6/157x4/377x4ほか計61)することを確認
= ICの取りこぼし・重複がないことの独立した裏づけ。

検証: 残存する74LSのValue 0件、変更行はValueの56行のみ
凍結マスターTB04addr8bitは08-23の状態で古いため対象外

Co-Authored-By: Claude Opus 5 <noreply@anthropic.com>
Parts:
- U901, U902, U903, U905: value 74LS377 -> 74HC377
Changed lines of the file:
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@@
 			)
 		)
-		(property "Value" "74LS377"
+		(property "Value" "74HC377"
 			(at 245.9833 167.64 0)
 			(show_name no)
@@
 			)
 		)
-		(property "Value" "74LS377"
+		(property "Value" "74HC377"
 			(at 242.1733 50.8 0)
 			(show_name no)
@@
 			)
 		)
-		(property "Value" "74LS377"
+		(property "Value" "74HC377"
 			(at 79.6133 52.07 0)
 			(show_name no)
@@
 			)
 		)
-		(property "Value" "74LS377"
+		(property "Value" "74HC377"
 			(at 83.4233 168.91 0)
 			(show_name no)
