File: ver2/hardware/基板分割_0827/TB04addr8bit_alu/TB04addr8bit_alu.kicad_sch (KiCad schematic)
At the start: 7 parts, among them J1602 Screw_Terminal_01x02, U102 74HC138

Commit message: ver2: 演算板からInterFaceシートを削除(命令表示は制御板へ)
- OPC/OPRは全部U602/U606の出力=制御板の信号なのでケーブル増設が不要に
- 階層ピン0を確認しトップシート・子ファイル・kicad_proの3点を整合削除
- 部品104→96、残るコネクタはJ601とJ1602のみ、パース確認済み

Co-Authored-By: Claude Opus 5 <noreply@anthropic.com>
Other:
- removed sheet InterFace
Changed lines of the file:
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@@
-	)
-	(sheet
-		(at 369.57 55.88)
-		(size 12.7 5.08)
-		(exclude_from_sim no)
-		(in_bom yes)
-		(on_board yes)
-		(dnp no)
-		(fields_autoplaced yes)
-		(stroke
-			(width 0.1524)
-			(type solid)
-		)
-		(fill
-			(color 0 0 0 0)
-		)
-		(property "Sheetname" "InterFace"
-			(at 369.57 55.1684 0)
-			(show_name no)
-			(do_not_autoplace no)
-			(effects
-				(font
-					(size 1.27 1.27)
-				)
-				(justify left bottom)
-			)
-		)
-		(property "Sheetfile" "ALU.kicad_sch"
-			(at 369.57 61.5446 0)
-			(show_name no)
-			(do_not_autoplace no)
-			(effects
-				(font
-					(size 1.27 1.27)
-				)
-				(justify left top)
-			)
-		)
-		(instances
-			(project "TB04addr4bitVer3"
-				(path "/4ea1f5c4-c9b0-4258-a3d4-23d6760fc0c5"
-					(page "6")
-				)
-			)
-			(project "TB04addr8bit_alu"
-				(path "/d176c79b-dced-4d01-bcec-7dfd676fcfc2"
-					(page "8")
-				)
-			)
-		)
 	)
 	(sheet

Commit message: ver2: 3分割にケーブル用・キャリア用コネクタを実装(検証全項目合格)
- ケーブル両端のピン割り当て100ピン全数一致、手順書の表とも不一致0
- またぐ47信号すべてコネクタに出ている(未接続0)
- isolated_pin_label 34→0、pin_not_driven 29→0

Co-Authored-By: Claude Opus 5 <noreply@anthropic.com>
Parts:
- added J2: Conn_02x20_Odd_Even, symbol Connector_Generic:Conn_02x20_Odd_Even
- added J3: Conn_02x10_Odd_Even, symbol Connector_Generic:Conn_02x10_Odd_Even
Connections:
- net DI0: now also J2.27 (Pin_27)
- net DI1: now also J2.25 (Pin_25)
- net DI2: now also J2.23 (Pin_23)
- net DI3: now also J2.21 (Pin_21)
- net EXE: now also J2.7 (Pin_7)
- net GND: now also J2.10 (Pin_10), J2.12 (Pin_12), J2.14 (Pin_14), J2.16 (Pin_16), J2.18 (Pin_18), J2.2 (Pin_2), J2.20 (Pin_20), J2.22 (Pin_22), J2.24 (Pin_24), J2.26 (Pin_26), J2.28 (Pin_28), J2.30 (Pin_30), J2.32 (Pin_32), J2.34 (Pin_34), J2.36 (Pin_36), J2.4 (Pin_4), J2.6 (Pin_6), J2.8 (Pin_8), J3.1 (Pin_1), J3.11 (Pin_11), J3.16 (Pin_16), J3.20 (Pin_20), J3.6 (Pin_6)
- net OPR4: now also J3.10 (Pin_10)
- net OPR5: now also J3.9 (Pin_9)
- net OPR6: now also J3.8 (Pin_8)
- net VDD: now also J2.38 (Pin_38), J2.40 (Pin_40)
- net sel_a0: now also J2.37 (Pin_37)
- net sel_a1: now also J2.35 (Pin_35)
- net sel_a2: now also J2.33 (Pin_33)
- net ~{Ena_RS01}: now also J3.18 (Pin_18)
- net ~{Enb_RS01}: now also J3.19 (Pin_19)
- net ~{WE}: now also J2.39 (Pin_39)
- new net CLK_C: J2.9 (Pin_9)
- new net CLK_CPU: J2.1 (Pin_1)
- new net CLK_Z: J2.11 (Pin_11)
- new net DCR: J2.5 (Pin_5)
- new net MD0: J2.19 (Pin_19)
- new net MD1: J2.17 (Pin_17)
- new net MD2: J2.15 (Pin_15)
- new net MD3: J2.13 (Pin_13)
- new net OPC0: J3.5 (Pin_5)
- new net OPC1: J3.4 (Pin_4)
- new net OPC2: J3.3 (Pin_3)
- new net OPC3: J3.2 (Pin_2)
- new net OPR0: J3.15 (Pin_15)
- new net OPR1: J3.14 (Pin_14)
- new net OPR2: J3.13 (Pin_13)
- new net OPR3: J3.12 (Pin_12)
- new net OPR7: J3.7 (Pin_7)
- new net SEL_IMM: J3.17 (Pin_17)
- new net carry_in: J2.29 (Pin_29)
- new net zero_prev: J2.31 (Pin_31)
- new net ~{RST}: J2.3 (Pin_3)

Commit message: ver2: 3分割のフットプリント設定完了・取付穴を追加・PCBを作り直し
- 新規コネクタ11件のフットプリントを設定(2x20/2x10ピンソケット・端子台)
- 演算板/制御板/キャリアに取付穴MountingHole_Pad×4とGNDを追加(M3・パッド付きビア)
- 3枚のPCBをコピー元マスターのレイアウトを一掃して作り直し(配置前・配線0)
- 階層から外れて残っていたRS00/RS01.kicad_sch(制御板・IF板)を削除

検証: フットプリント未設定0件、回路図とPCBの参照番号の集合差分0
(演算102/制御101/IF127/キャリア14)、回路図の電気的変更なし

Co-Authored-By: Claude Opus 5 <noreply@anthropic.com>
Parts:
- added H101, H102, H103, H104: MountingHole_Pad, MountingHole:MountingHole_3.2mm_M3_Pad_Via, symbol Mechanical:MountingHole_Pad
- J1602: footprint (none) -> TerminalBlock:TerminalBlock_MaiXu_MX126-5.0-02P_1x02_P5.00mm
- J2: footprint (none) -> Connector_PinSocket_2.54mm:PinSocket_2x20_P2.54mm_Vertical
- J3: footprint (none) -> Connector_PinSocket_2.54mm:PinSocket_2x10_P2.54mm_Vertical
Connections:
- net GND: now also H101.1, H102.1, H103.1, H104.1
