File: ver2/hardware/基板分割_0827/TB04addr8bit_alu/Decoder.kicad_sch (KiCad schematic)
At the start: 12 parts, among them U701 74LS273, U702 74LS273, U703 28C256, U704 28C256, U705 74LS273, U706 28C256

Commit message: ver2: 3分割で他基板側のICを削除(ctrl 9・alu 15・if 2個)
削除前にまたぎ本数(37/20)で割り当てを検算。kicad-cliのパース通過を確認。

Co-Authored-By: Claude Opus 5 <noreply@anthropic.com>
Parts:
- removed U701, U705: 74LS273, Package_DIP:DIP-20_W7.62mm_Socket, symbol 74xx:74LS273
- removed U703, U706: 28C256, Package_DIP:DIP-28_W15.24mm_Socket, symbol Memory_EEPROM:28C256

Commit message: ver2: 3分割でシート内の不要部品・配線を削除(検証合格)／キャリアを0827へコピー
- 制御34・演算25・IF10=IC69でマスターと一致、部品の取りこぼし0
- ピン-ネット署名の変化0件=誤って線を切った箇所なし
- またぐ信号は制御/演算35・IF/制御18で手順書の表と過不足ゼロ

Co-Authored-By: Claude Opus 5 <noreply@anthropic.com>
Parts:
- removed C701, C702, C705, C706: 0.1u, Capacitor_THT:C_Disc_D4.3mm_W1.9mm_P5.00mm, symbol Device:C
Connections:
- no-connect marks 2 -> 0

Commit message: ver2: 3分割の74LS表記をHCへ一括変更(31パッケージ・Valueのみ)
- 書き換えたのはValueプロパティのみ(56件=31パッケージ)
- lib_id(74xx:74LS***)とDatasheetは変更せず。HC品のシンボルがKiCADに
  無いため、lib_idを変えるとシンボル未検出になる
- 74LS->74HCの単純置換で9品種すべて実在の型番(00/08/10/32/139/157/
  253/273/377)。ピン配置は同一でネットリストへの影響なし

検証: 残存する74LSのValue 0件、git diffの変更行はValueの56行のみ
申し送り: PCB側のValueは未同期。「回路図からPCBを更新」で解消する

Co-Authored-By: Claude Opus 5 <noreply@anthropic.com>
Parts:
- U702: value 74LS273 -> 74HC273
Changed lines of the file:
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@@
 			)
 		)
-		(property "Value" "74LS273"
+		(property "Value" "74HC273"
 			(at 148.1933 57.15 0)
 			(show_name no)
