File: ver2/hardware/基板分割_0827/TB04addr8bit_alu/RS00.kicad_sch (KiCad schematic)
At the start: 34 parts, among them IC201 74HC161N, IC202 74HC161N, IC203 74HC161N, IC204 74HC161N, U201 74LS253, U202 74LS253, U203 74LS253, U204 74LS253

Commit message: ver2: 3分割の74LS表記をHCへ一括変更(31パッケージ・Valueのみ)
- 書き換えたのはValueプロパティのみ(56件=31パッケージ)
- lib_id(74xx:74LS***)とDatasheetは変更せず。HC品のシンボルがKiCADに
  無いため、lib_idを変えるとシンボル未検出になる
- 74LS->74HCの単純置換で9品種すべて実在の型番(00/08/10/32/139/157/
  253/273/377)。ピン配置は同一でネットリストへの影響なし

検証: 残存する74LSのValue 0件、git diffの変更行はValueの56行のみ
申し送り: PCB側のValueは未同期。「回路図からPCBを更新」で解消する

Co-Authored-By: Claude Opus 5 <noreply@anthropic.com>
Parts:
- U201, U202, U203, U204: value 74LS253 -> 74HC253
Changed lines of the file:
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@@
 			)
 		)
-		(property "Value" "74LS253"
+		(property "Value" "74HC253"
 			(at 327.2633 99.06 0)
 			(show_name no)
@@
 			)
 		)
-		(property "Value" "74LS253"
+		(property "Value" "74HC253"
 			(at 262.4933 144.78 0)
 			(show_name no)
@@
 			)
 		)
-		(property "Value" "74LS253"
+		(property "Value" "74HC253"
 			(at 294.2433 217.17 0)
 			(show_name no)
@@
 			)
 		)
-		(property "Value" "74LS253"
+		(property "Value" "74HC253"
 			(at 327.2633 21.59 0)
 			(show_name no)
