File: ver2/hardware/基板分割_0827/TB04addr8bit_alu/RS00.kicad_sch (KiCad schematic)
At the start: 34 parts, among them IC201 74HC161N, IC202 74HC161N, IC203 74HC161N, IC204 74HC161N, U201 74HC253, U202 74HC253, U203 74HC253, U204 74HC253

Commit message: ver2: 3枚の外形を高さ150mmに統一／制御板のプルダウンをSIP集約・取付穴2個追加(配置は途中)
- 外形: 演算130x150・制御200x150・IF135x150
- 制御板: R603-R606(10K x4)をRN602(R_Array_SIP5)へ集約／取付穴H105・H106を追加／U1101のフットプリントをDIP-24_W15.24mm_Socketへ
- 検証: 署名変化は制御8ピン(ネット名のみ・構成員同一)と演算32ピン(同値素子の割り当て替え)だけ／未接続入力0・単一構成員ネット0・回路図とPCBの参照番号差分0
Connections:
- net at D205.1 (K): now also RN201.8 (R7); no longer RN201.4 (R3)
- net at D208.1 (K): now also RN202.9 (R8); no longer RN202.5 (R4)
- net at D216.1 (K): now also RN202.5 (R4); no longer RN202.9 (R8)
- net at D215.1 (K): now also RN201.5 (R4); no longer RN201.9 (R8)
- net at D204.1 (K): now also RN202.7 (R6); no longer RN202.3 (R2)
- net at D207.1 (K): now also RN201.9 (R8); no longer RN201.5 (R4)
- net at D201.1 (K): now also RN201.6 (R5); no longer RN201.2 (R1)
- net at D214.1 (K): now also RN202.4 (R3); no longer RN202.8 (R7)
- net at D211.1 (K): now also RN201.3 (R2); no longer RN201.7 (R6)
- net at D209.1 (K): now also RN201.2 (R1); no longer RN201.6 (R5)
- net at D210.1 (K): now also RN202.2 (R1); no longer RN202.6 (R5)
- net at D202.1 (K): now also RN202.6 (R5); no longer RN202.2 (R1)
- net at D203.1 (K): now also RN201.7 (R6); no longer RN201.3 (R2)
- net at D206.1 (K): now also RN202.8 (R7); no longer RN202.4 (R3)
- net at D212.1 (K): now also RN202.3 (R2); no longer RN202.7 (R6)
- net at D213.1 (K): now also RN201.4 (R3); no longer RN201.8 (R7)
