File: ver2/hardware/基板分割_0827/TB04addr8bit_alu/TB04addr8bit_alu.kicad_pcb (KiCad board)
At the start: 2 copper layers, 295 x 195 mm, 307 parts, among them IC201 74HC161N, IC202 74HC161N, IC203 74HC161N, IC204 74HC161N, IC301 74HC161N, IC302 74HC161N, IC303 74HC161N, IC304 74HC161N, IC401 74HC161N, IC402 74HC161N, IC601 74HC161N, J1001 Conn_01x06_Socket, J1002 Conn_01x06_Socket, J1003 Conn_01x06_Socket, J1004 Conn_01x06_Socket, J101 USB_C_Receptacle_PowerOnly_6P, J601 Conn_02x05_Odd_Even, J801 Conn_02x05_Odd_Even, J802 Conn_02x05_Odd_Even, J803 Conn_02x05_Odd_Even, J804 Conn_02x05_Odd_Even, J805 Conn_02x05_Odd_Even, J806 Conn_02x05_Odd_Even, J807 Conn_02x05_Odd_Even, J808 Conn_02x05_Odd_Even, J901 Conn_02x05_Odd_Even, J902 Conn_02x05_Odd_Even, J903 Conn_02x05_Odd_Even, J904 Conn_02x05_Odd_Even, SW1001 SW_DIP_x04, SW1002 SW_DIP_x04, SW1003 SW_DIP_x04, SW1004 SW_DIP_x04, SW101 SW_SPDT, SW501 SW_Push, SW502 sw rotary, SW503 SW_Push, SW601 SW_Coded_SH-7050, U1001 74HC244, U1002 74HC244, U1003 74HC244, U1004 74HC244, U101 74LS157, U102 74HC138, U1101 6116, U1102 74HC244, U1103 74HC244, U1201 74HC193, U1301 74LS08, U1401 74HC138, U1402 74HC244, U1403 74HC244, U1404 74HC244, U1405 74HC244, U1406 74LS157, U1407 74LS139, U1501 74AHC04, U1503 74LS08, U1504 74HC00, U1505 74LS00, U1506 74LS32, U1507 74LS08, U1509 74LS10, U201 74LS253, U202 74LS253, U203 74LS253, U204 74LS253, U301 74LS253, U302 74LS253, U303 74LS253, U304 74LS253, U401 74LS157, U402 74LS253, U403 74LS253, U404 74LS157, U405 74LS253, U406 74LS253, U501 74HC14, U502 4060, U601 74LS273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

Commit message: ver2: 3分割のフットプリント設定完了・取付穴を追加・PCBを作り直し
- 新規コネクタ11件のフットプリントを設定(2x20/2x10ピンソケット・端子台)
- 演算板/制御板/キャリアに取付穴MountingHole_Pad×4とGNDを追加(M3・パッド付きビア)
- 3枚のPCBをコピー元マスターのレイアウトを一掃して作り直し(配置前・配線0)
- 階層から外れて残っていたRS00/RS01.kicad_sch(制御板・IF板)を削除

検証: フットプリント未設定0件、回路図とPCBの参照番号の集合差分0
(演算102/制御101/IF127/キャリア14)、回路図の電気的変更なし

Co-Authored-By: Claude Opus 5 <noreply@anthropic.com>
Parts:
- removed C1001, C1002, C1003, C1004, C101, C1101, C1102, C1103, C1201, C1301, C1401, C1402, C1403, C1404, C1407, C1408, C1409, C1501, C1502, C1503, C1504, C1505, C1506, C1507, C401, C402, C403, C404, C503, C504, C602, C603, C604, C605, C606, C607, C701, C702, C705, C706, C901, C902, C903, C904: 0.1u, Capacitor_THT:C_Disc_D4.3mm_W1.9mm_P5.00mm
- removed C501, C502: 10u 16V, Capacitor_THT:CP_Radial_D5.0mm_P2.00mm
- removed C505, C506: 22p, Capacitor_THT:C_Disc_D4.3mm_W1.9mm_P5.00mm
- removed D1001, D1002, D1003, D1004, D1005, D1006, D1007, D1008, D1009, D1010, D1011, D1012, D1013, D1014, D1015, D1016, D1201, D1202, D1203, D501, D502, D603, D604, D605, D606, D901, D902, D903, D904, D905, D906, D907, D908, D909, D910, D911, D912, D913, D914, D915, D916: LED, LED_THT:LED_D3.0mm_Clear
- removed H501, H502, H503, H504: MountingHole_Pad, MountingHole:MountingHole_3.2mm_M3_Pad_Via
- removed IC401, IC402, IC601: 74HC161N, Package_DIP:DIP-16_W7.62mm_Socket
- removed J1001, J1002, J1003, J1004: Conn_01x06_Socket, Connector_PinSocket_2.54mm:PinSocket_1x06_P2.54mm_Vertical
- removed J101: USB_C_Receptacle_PowerOnly_6P, Library:USB_C_receptacle_onlypower_tanuki
- removed J801, J802, J803, J804, J805, J806, J807, J808, J901, J902, J903, J904: Conn_02x05_Odd_Even, Connector_PinSocket_2.54mm:PinSocket_2x05_P2.54mm_Vertical
- removed R1001, R1002, R1003, R1004, R1005, R1006, R1007, R1008, R1009, R1010, R1011, R1012, R1013, R1014, R1015, R1016, R501, R502: 1K, Resistor_THT:R_Axial_DIN0207_L6.3mm_D2.5mm_P10.16mm_Horizontal
- removed R101, R102: 5.1K, Resistor_THT:R_Axial_DIN0207_L6.3mm_D2.5mm_P10.16mm_Horizontal
- removed R1201, R1202, R1203: 4.7K, Resistor_THT:R_Axial_DIN0207_L6.3mm_D2.5mm_P10.16mm_Horizontal
- removed R503, R506, R603, R604, R605, R606: 10K, Resistor_THT:R_Axial_DIN0207_L6.3mm_D2.5mm_P10.16mm_Horizontal
- removed R504, R507, R509: 100K, Resistor_THT:R_Axial_DIN0207_L6.3mm_D2.5mm_P7.62mm_Horizontal
- removed R505: 100, Resistor_THT:R_Axial_DIN0207_L6.3mm_D2.5mm_P10.16mm_Horizontal
- removed R508, R510: 3.3K, Resistor_THT:R_Axial_DIN0207_L6.3mm_D2.5mm_P7.62mm_Horizontal
- removed R511: 10M, Resistor_THT:R_Axial_DIN0207_L6.3mm_D2.5mm_P10.16mm_Horizontal
- removed R512: 220K, Resistor_THT:R_Axial_DIN0207_L6.3mm_D2.5mm_P10.16mm_Horizontal
- removed RN1002, RN1003, RN1005, RN1007, RN601, RN901, RN902, RN903, RN904: 4.7K, Resistor_THT:R_Array_SIP5
- removed RN1009, RN1010: 47K, Resistor_THT:R_Array_SIP9
- removed SW1001, SW1002, SW1003, SW1004: SW_DIP_x04, Button_Switch_THT:SW_DIP_SPSTx04_Slide_9.78x12.34mm_W7.62mm_P2.54mm
- removed SW101: SW_SPDT, Library:sw_slide
- removed SW501, SW503: SW_Push, Button_Switch_THT:SW_Tactile_Straight_KSL0Axx1LFTR
- removed SW502: sw rotary, LibraryTB04:SW_Rotary_1x9_Alpha_SR1712F-0109
- removed SW601: SW_Coded_SH-7050, Library:dip_rotary_sw
- removed U1001, U1002, U1003, U1004, U1102, U1103, U1402, U1403, U1404, U1405: 74HC244, Package_DIP:DIP-20_W7.62mm_Socket
- removed U101, U1406, U401, U404: 74LS157, Package_DIP:DIP-16_W7.62mm_Socket
- removed U1101: 6116, Package_DIP:DIP-24_18.0mmx34.29mm_W15.24mm_Socket
- removed U1201: 74HC193, Package_DIP:DIP-16_W7.62mm_Socket
- removed U1301, U1503, U1507: 74LS08, Package_DIP:DIP-14_W7.62mm_Socket
- removed U1401: 74HC138, Package_DIP:DIP-16_W7.62mm_Socket
- removed U1407: 74LS139, Package_DIP:DIP-16_W7.62mm_Socket
- removed U1501: 74AHC04, Package_DIP:DIP-14_W7.62mm_Socket
- removed U1504: 74HC00, Package_DIP:DIP-14_W7.62mm_Socket
- removed U1505: 74LS00, Package_DIP:DIP-14_W7.62mm_Socket
- removed U1506: 74LS32, Package_DIP:DIP-14_W7.62mm_Socket
- removed U1509: 74LS10, Package_DIP:DIP-14_W7.62mm_Socket
- removed U501: 74HC14, Package_DIP:DIP-14_W7.62mm_Socket
- removed U502: 4060, Package_DIP:DIP-16_W7.62mm_Socket
- removed U601, U701, U705: 74LS273, Package_DIP:DIP-20_W7.62mm_Socket
- removed U602, U606: 74HC273, Package_DIP:DIP-20_W7.62mm_Socket
- removed U604: 28C256, Socket:DIP_Socket-28_W11.9mm_W12.7mm_W15.24mm_W17.78mm_W18.5mm_3M_228-1277-00-0602J
- removed U607: 74HC238, Package_DIP:DIP-16_W7.62mm_Socket
- removed U703, U706: 28C256, Package_DIP:DIP-28_W15.24mm_Socket
- removed U901, U902, U903, U905: 74LS377, Package_DIP:DIP-20_W7.62mm_Socket
- removed Y501: 32.768KHz, Connector_PinSocket_2.00mm:PinSocket_1x02_P2.00mm_Vertical
- added H101: MountingHole_Pad, MountingHole:MountingHole_3.2mm_M3_Pad_Via, F.Cu at (273.5, 188.5)
- added H102: MountingHole_Pad, MountingHole:MountingHole_3.2mm_M3_Pad_Via, F.Cu at (273.5, 196.4)
- added H103: MountingHole_Pad, MountingHole:MountingHole_3.2mm_M3_Pad_Via, F.Cu at (273.5, 204.4)
- added H104: MountingHole_Pad, MountingHole:MountingHole_3.2mm_M3_Pad_Via, F.Cu at (273.5, 212.3)
- added J1602: Screw_Terminal_01x02, TerminalBlock:TerminalBlock_MaiXu_MX126-5.0-02P_1x02_P5.00mm, F.Cu at (346.5, 132.6)
- added J2: Conn_02x20_Odd_Even, Connector_PinSocket_2.54mm:PinSocket_2x20_P2.54mm_Vertical, F.Cu at (340.2, 102.4)
- added J3: Conn_02x10_Odd_Even, Connector_PinSocket_2.54mm:PinSocket_2x10_P2.54mm_Vertical, F.Cu at (347.3, 102.4)
- moved U702 297.6 mm to (356.8, 50.6), turned to 0 degrees
- moved U704 282.7 mm to (337.4, 50.6), turned to 0 degrees
- moved C704 277.9 mm to (356.3, 80.8), turned to 0 degrees
- moved U204 258.6 mm to (323.7, 102.2), turned to 0 degrees
- moved C601 257.5 mm to (316.6, 181.0), turned to 0 degrees
- moved C703 248.0 mm to (356.3, 77.3), turned to 0 degrees
- moved C608 237.4 mm to (316.6, 184.4), turned to 0 degrees
- moved U202 233.5 mm to (300.3, 102.2), turned to 0 degrees
- moved C102 228.8 mm to (344.1, 143.4), turned to 0 degrees
- moved U102 223.0 mm to (351.7, 102.2), turned to 0 degrees
- moved U203 222.4 mm to (312.0, 102.2), turned to 0 degrees
- moved D214 221.9 mm to (291.7, 130.3)
- moved D212 220.6 mm to (285.9, 141.2)
- moved D215 215.3 mm to (291.7, 135.8)
- moved D211 197.7 mm to (285.9, 135.8)
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Other:
- board size 295 x 195 mm -> 125 x 135 mm

Commit message: ver2: 制御板の配置を差し戻し(外形200x135へ復帰)・J5を削除
- 外形を200x180に変えたのは行き過ぎだったため、配置ごと
  fb4b7f8の状態へ戻した(演算板が上に載る機械的制約を
  考慮していなかった)
- 回路図で削除済みのJ5(キャリア用2x10)をPCBからも削除

Co-Authored-By: Claude Opus 5 <noreply@anthropic.com>
Parts:
- U201, U202, U203, U204, U301, U302, U303, U304, U402, U403, U405, U406: value 74LS253 -> 74HC253
- U702: value 74LS273 -> 74HC273
Changed lines of the file:
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@@
 			)
 		)
-		(property "Value" "74LS253"
+		(property "Value" "74HC253"
 			(at 3.81 20.11 0)
 			(layer "F.Fab")
@@
 			)
 		)
-		(property "Value" "74LS253"
+		(property "Value" "74HC253"
 			(at 3.81 20.11 0)
 			(layer "F.Fab")
@@
 			)
 		)
-		(property "Value" "74LS253"
+		(property "Value" "74HC253"
 			(at 3.81 20.11 0)
 			(layer "F.Fab")
@@
 			)
 		)
-		(property "Value" "74LS253"
+		(property "Value" "74HC253"
 			(at 3.81 20.11 0)
 			(layer "F.Fab")
@@
 			)
 		)
-		(property "Value" "74LS253"
+		(property "Value" "74HC253"
 			(at 3.81 20.11 0)
 			(layer "F.Fab")
@@
 			)
 		)
-		(property "Value" "74LS253"
+		(property "Value" "74HC253"
 			(at 3.81 20.11 0)
 			(layer "F.Fab")
@@
 			)
 		)
-		(property "Value" "74LS253"
+		(property "Value" "74HC253"
 			(at 3.81 20.11 0)
 			(layer "F.Fab")
@@
 			)
 		)
-		(property "Value" "74LS253"
+		(property "Value" "74HC253"
 			(at 3.81 20.11 0)
 			(layer "F.Fab")
@@
 			)
 		)
-		(property "Value" "74LS253"
+		(property "Value" "74HC253"
 			(at 3.81 20.11 0)
 			(layer "F.Fab")
@@
 			)
 		)
-		(property "Value" "74LS273"
+		(property "Value" "74HC273"
 			(at 3.81 25.19 0)
 			(layer "F.Fab")
@@
 			)
 		)
-		(property "Value" "74LS253"
+		(property "Value" "74HC253"
 			(at 3.81 20.11 0)
 			(layer "F.Fab")
@@
 			)
 		)
-		(property "Value" "74LS253"
+		(property "Value" "74HC253"
 			(at 3.81 20.11 0)
 			(layer "F.Fab")
@@
 			)
 		)
-		(property "Value" "74LS253"
+		(property "Value" "74HC253"
 			(at 3.81 20.11 0)
 			(layer "F.Fab")

Commit message: ver2: 演算板の部品配置を更新／RS01回路図の配線を整理
外形125x135。102部品のうち62部品を外形内に配置。
courtyard重なり0。配線は未着手。

Co-Authored-By: Claude Opus 5 <noreply@anthropic.com>
Claude-Session: https://claude.ai/code/session_01AfeTYjKzCvUCekJLNec6bd
Parts:
- moved H101 214.9 mm to (105.0, 55.0)
- moved U301 178.7 mm to (111.0, 70.6), turned to 90 degrees
- moved U201 177.6 mm to (111.5, 115.9), turned to 90 degrees
- moved D310 175.0 mm to (112.0, 58.5), turned to 90 degrees
- moved D312 170.7 mm to (118.0, 58.5), turned to 90 degrees
- moved H102 169.3 mm to (105.0, 180.0)
- moved D314 168.9 mm to (124.0, 58.5), turned to 90 degrees
- moved H104 166.2 mm to (220.0, 55.0)
- moved D316 164.7 mm to (130.0, 58.5), turned to 90 degrees
- moved U302 163.9 mm to (137.6, 70.7), turned to 90 degrees
- moved U202 163.1 mm to (137.8, 116.2), turned to 90 degrees
- moved U203 148.7 mm to (164.0, 116.6), turned to 90 degrees
- moved U303 147.8 mm to (165.5, 70.2), turned to 90 degrees
- moved IC204 138.4 mm to (151.8, 161.3), turned to 90 degrees
- moved D302 137.6 mm to (138.0, 58.5), turned to 90 degrees
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Connections:
- RN301 pad 2: Net-(D301-K) -> Net-(D309-K)
- RN301 pad 3: Net-(D303-K) -> Net-(D311-K)
- RN301 pad 4: Net-(D305-K) -> Net-(D313-K)
- RN301 pad 5: Net-(D307-K) -> Net-(D315-K)
- RN301 pad 6: Net-(D309-K) -> Net-(D301-K)
- RN301 pad 7: Net-(D311-K) -> Net-(D303-K)
- RN301 pad 8: Net-(D313-K) -> Net-(D305-K)
- RN301 pad 9: Net-(D315-K) -> Net-(D307-K)
- RN302 pad 2: Net-(D302-K) -> Net-(D310-K)
- RN302 pad 3: Net-(D304-K) -> Net-(D312-K)
- RN302 pad 4: Net-(D306-K) -> Net-(D314-K)
- RN302 pad 5: Net-(D308-K) -> Net-(D316-K)
- RN302 pad 6: Net-(D310-K) -> Net-(D302-K)
- RN302 pad 7: Net-(D312-K) -> Net-(D304-K)
- RN302 pad 8: Net-(D314-K) -> Net-(D306-K)
- RN302 pad 9: Net-(D316-K) -> Net-(D308-K)
