File: ver2/hardware/基板分割_0827/TB04addr8bit_ctrl/AddrDecord.kicad_sch (KiCad schematic)
At the start: 2 parts, among them U1301 74LS08

Commit message: ver2: 3分割の74LS表記をHCへ一括変更(31パッケージ・Valueのみ)
- 書き換えたのはValueプロパティのみ(56件=31パッケージ)
- lib_id(74xx:74LS***)とDatasheetは変更せず。HC品のシンボルがKiCADに
  無いため、lib_idを変えるとシンボル未検出になる
- 74LS->74HCの単純置換で9品種すべて実在の型番(00/08/10/32/139/157/
  253/273/377)。ピン配置は同一でネットリストへの影響なし

検証: 残存する74LSのValue 0件、git diffの変更行はValueの56行のみ
申し送り: PCB側のValueは未同期。「回路図からPCBを更新」で解消する

Co-Authored-By: Claude Opus 5 <noreply@anthropic.com>
Parts:
- U1301: value 74LS08 -> 74HC08
Changed lines of the file:
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@@
 			)
 		)
-		(property "Value" "74LS08"
+		(property "Value" "74HC08"
 			(at 67.3017 55.88 0)
 			(show_name no)
@@
 			)
 		)
-		(property "Value" "74LS08"
+		(property "Value" "74HC08"
 			(at 119.3717 60.96 0)
 			(show_name no)
@@
 			)
 		)
-		(property "Value" "74LS08"
+		(property "Value" "74HC08"
 			(at 92.7017 53.34 0)
 			(show_name no)
@@
 			)
 		)
-		(property "Value" "74LS08"
+		(property "Value" "74HC08"
 			(at 114.3 114.2999 0)
 			(show_name no)
@@
 			)
 		)
-		(property "Value" "74LS08"
+		(property "Value" "74HC08"
 			(at 67.3017 34.29 0)
 			(show_name no)
