File: ver2/hardware/基板分割_0827/TB04addr8bit_ctrl/ram.kicad_sch (KiCad schematic)
At the start: 6 parts, among them U1101 6116, U1102 74HC244, U1103 74HC244

Commit message: ver2: 3枚の外形を高さ150mmに統一／制御板のプルダウンをSIP集約・取付穴2個追加(配置は途中)
- 外形: 演算130x150・制御200x150・IF135x150
- 制御板: R603-R606(10K x4)をRN602(R_Array_SIP5)へ集約／取付穴H105・H106を追加／U1101のフットプリントをDIP-24_W15.24mm_Socketへ
- 検証: 署名変化は制御8ピン(ネット名のみ・構成員同一)と演算32ピン(同値素子の割り当て替え)だけ／未接続入力0・単一構成員ネット0・回路図とPCBの参照番号差分0
Parts:
- U1101: footprint Package_DIP:DIP-24_18.0mmx34.29mm_W15.24mm_Socket -> Package_DIP:DIP-24_W15.24mm_Socket
Changed lines of the file:
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@@
 			)
 		)
-		(property "Footprint" "Package_DIP:DIP-24_18.0mmx34.29mm_W15.24mm_Socket"
+		(property "Footprint" "Package_DIP:DIP-24_W15.24mm_Socket"
 			(at 77.47 44.45 0)
 			(hide yes)
