File: ver2/hardware/基板分割_0827/TB04addr8bit_ctrl/TB04addr8bit_ctrl.kicad_pcb (KiCad board)
At the start: 2 copper layers, 210 x 170 mm, 101 parts, among them IC401 74HC161N, IC402 74HC161N, IC601 74HC161N, J1 Conn_02x20_Odd_Even, J1602 Screw_Terminal_01x02, J2 Conn_02x20_Odd_Even, J3 Conn_02x10_Odd_Even, J6 Conn_02x05_Odd_Even, J7 Conn_02x05_Odd_Even, J8 Conn_02x05_Odd_Even, J801 Conn_02x05_Odd_Even, J802 Conn_02x05_Odd_Even, J803 Conn_02x05_Odd_Even, J804 Conn_02x05_Odd_Even, J9 Conn_02x05_Odd_Even, SW601 SW_Coded_SH-7050, U101 74HC157, U1101 6116, U1102 74HC244, U1103 74HC244, U1201 74HC193, U1301 74HC08, U1401 74HC138, U1402 74HC244, U1403 74HC244, U1404 74HC244, U1405 74HC244, U1406 74HC157, U1407 74HC139, U1501 74AHC04, U1503 74HC08, U1504 74HC00, U1505 74HC00, U1506 74HC32, U1509 74HC10, U401 74HC157, U404 74HC157, U601 74HC273, U602 74HC273, U604 28C256, U606 74HC273, U607 74HC238, U701 74HC273, U703 28C256, U705 74HC273, U706 28C256

Commit message: ver2: 制御板のGND以外の配線が完了(DRC 0件・残りはGND 185)
Co-Authored-By: Claude Opus 5 <noreply@anthropic.com>
Routing:
- net ~{WE_RAM}: track 0.00 -> 66.9 mm, vias 0 -> 1
- net Net-(IC601-Q1): track 0.00 -> 27.2 mm
- net GND: track 0.00 -> 23.5 mm
- net Net-(D101-A): track 0.00 -> 22.8 mm
- net Net-(IC601-Q0): track 0.00 -> 21.2 mm
- net VDD: track 1359.2 -> 1366.0 mm, vias 10 -> 12
Changed lines of the file:
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@@
 	)
 	(segment
+		(start 136.06 115.885)
+		(end 140.92 115.885)
+		(width 0.5)
+		(layer "F.Cu")
+		(net "GND")
+	)
+	(segment
+		(start 152.38 120.885)
+		(end 157.46 120.885)
+		(width 0.5)
+		(layer "F.Cu")
+		(net "GND")
+	)
+	(segment
+		(start 140.92 115.885)
+		(end 143.3 118.265)
+		(width 0.5)
+		(layer "F.Cu")
+		(net "GND")
+	)
+	(segment
+		(start 143.3 118.265)
+		(end 149.76 118.265)
+		(width 0.5)
+		(layer "F.Cu")
+		(net "GND")
+	)
+	(segment
+		(start 149.76 118.265)
+		(end 152.38 120.885)
+		(width 0.5)
+		(layer "F.Cu")
+		(net "GND")
+	)
+	(segment
 		(start 161.5 209)
 		(end 159.84 209)
@@
 	)
 	(segment
+		(start 141.14 111.105)
+		(end 135.195 111.105)
+		(width 0.8)
+		(layer "F.Cu")
+		(net "VDD")
+	)
+	(segment
 		(start 158.295 152.2)
 		(end 209.1 152.2)
@@
 	)
 	(segment
+		(start 134.5 113.13401)
+		(end 132.33401 115.3)
+		(width 0.8)
+		(layer "F.Cu")
+		(net "VDD")
+	)
+	(segment
 		(start 253.98 148.825)
 		(end 249.98 148.825)
@@
 	)
 	(segment
+		(start 134.5 111.8)
+		(end 134.5 113.13401)
+		(width 0.8)
+		(layer "F.Cu")
+		(net "VDD")
+	)
+	(segment
 		(start 268.08 111.865)
 		(end 270.36 111.865)
@@
 	)
 	(segment
+		(start 135.195 111.105)
+		(end 134.5 111.8)
+		(width 0.8)
+		(layer "F.Cu")
+		(net "VDD")
+	)
+	(segment
 		(start 249.835 113.265)
 		(end 247.4 115.7)
@@
 	)
 	(segment
-		(start 136.06 120.885)
-		(end 143.3 113.645)
-		(width 0.8)
-		(layer "F.Cu")
-		(net "VDD")
-	)
-	(segment
 		(start 114.28 120.885)
 		(end 116.82 120.885)
@@
 	)
 	(via
+		(at 141.14 111.105)
+		(size 0.8)
+		(drill 0.4)
+		(layers "F.Cu" "B.Cu")
+		(net "VDD")
+	)
+	(via
 		(at 214.42 147.28)
 		(size 0.8)
@@
 	)
 	(via
+		(at 132.33401 115.3)
+		(size 0.8)
+		(drill 0.4)
+		(layers "F.Cu" "B.Cu")
+		(net "VDD")
+	)
+	(via
 		(at 241.2 129.645)
 		(size 0.8)
@@
 	)
 	(segment
+		(start 132.33401 115.3)
+		(end 132.33401 120.61099)
+		(width 0.8)
+		(layer "B.Cu")
+		(net "VDD")
+	)
+	(segment
 		(start 279.066493 172.45)
 		(end 279.066493 189.573097)
@@
 	)
 	(segment
+		(start 132.33401 120.61099)
+		(end 132.06 120.885)
+		(width 0.8)
+		(layer "B.Cu")
+		(net "VDD")
+	)
+	(segment
 		(start 185.4 181.785)
 		(end 185.4 176.47401)
@@
 	)
 	(segment
+		(start 128.08 121.985)
+		(end 126.98 120.885)
+		(width 0.2)
+		(layer "F.Cu")
+		(net "Net-(IC601-Q0)")
+	)
+	(segment
+		(start 146.2 121.985)
+		(end 128.08 121.985)
+		(width 0.2)
+		(layer "F.Cu")
+		(net "Net-(IC601-Q0)")
+	)
+	(segment
+		(start 147.3 120.885)
+		(end 146.2 121.985)
+		(width 0.2)
+		(layer "F.Cu")
+		(net "Net-(IC601-Q0)")
+	)
+	(segment
+		(start 144.9 120.9)
+		(end 138.5 120.9)
+		(width 0.2)
+		(layer "F.Cu")
+		(net "Net-(IC601-Q1)")
+	)
+	(segment
+		(start 146.015 119.785)
+		(end 144.9 120.9)
+		(width 0.2)
+		(layer "F.Cu")
+		(net "Net-(IC601-Q1)")
+	)
+	(segment
+		(start 149.84 120.885)
+		(end 148.74 119.785)
+		(width 0.2)
+		(layer "F.Cu")
+		(net "Net-(IC601-Q1)")
+	)
+	(segment
+		(start 138.5 120.9)
+		(end 137.385 119.785)
+		(width 0.2)
+		(layer "F.Cu")
+		(net "Net-(IC601-Q1)")
+	)
+	(segment
+		(start 137.385 119.785)
+		(end 125.54 119.785)
+		(width 0.2)
+		(layer "F.Cu")
+		(net "Net-(IC601-Q1)")
+	)
+	(segment
+		(start 148.74 119.785)
+		(end 146.015 119.785)
+		(width 0.2)
+		(layer "F.Cu")
+		(net "Net-(IC601-Q1)")
+	)
+	(segment
+		(start 125.54 119.785)
+		(end 124.44 120.885)
+		(width 0.2)
+		(layer "F.Cu")
+		(net "Net-(IC601-Q1)")
+	)
+	(segment
 		(start 147.730304 191.2)
 		(end 138.5 191.2)
@@
 	)
 	(segment
+		(start 240.95 58.55)
+		(end 241.3 58.9)
+		(width 0.2)
+		(layer "F.Cu")
+		(net "~{WE_RAM}")
+	)
+	(segment
+		(start 180.32 60.265)
+		(end 182.035 58.55)
+		(width 0.2)
+		(layer "F.Cu")
+		(net "~{WE_RAM}")
+	)
+	(segment
+		(start 182.035 58.55)
+		(end 240.95 58.55)
+		(width 0.2)
+		(layer "F.Cu")
+		(net "~{WE_RAM}")
+	)
+	(via
+		(at 241.3 58.9)
+		(size 0.6)
+		(drill 0.3)
+		(layers "F.Cu" "B.Cu")
+		(net "~{WE_RAM}")
+	)
+	(segment
+		(start 241.82 59.42)
+		(end 241.82 63.765)
+		(width 0.2)
+		(layer "B.Cu")
+		(net "~{WE_RAM}")
+	)
+	(segment
+		(start 241.3 58.9)
+		(end 241.82 59.42)
+		(width 0.2)
+		(layer "B.Cu")
+		(net "~{WE_RAM}")
+	)
+	(segment
 		(start 213.6 124.5)
 		(end 213.7 124.4)
@@
 	)
 	(segment
+		(start 308 198.459999)
+		(end 308 180)
+		(width 0.25)
+		(layer "F.Cu")
+		(net "Net-(D101-A)")
+	)
+	(segment
+		(start 304.96 201.499999)
+		(end 308 198.459999)
+		(width 0.25)
+		(layer "F.Cu")
+		(net "Net-(D101-A)")
+	)
+	(segment
