File: ver2/hardware/基板分割_0827/TB04addr8bit_if/inPut.kicad_sch (KiCad schematic)
At the start: 54 parts, among them J1001 Conn_01x06_Socket, J1002 Conn_01x06_Socket, J1003 Conn_01x06_Socket, J1004 Conn_01x06_Socket, SW1001 SW_DIP_x04, SW1002 SW_DIP_x04, SW1003 SW_DIP_x04, SW1004 SW_DIP_x04, U1001 74HC244, U1002 74HC244, U1003 74HC244, U1004 74HC244

Commit message: ver2: inPortのプルダウンを47K→10Kへ(RN1009/RN1010のValueのみ32件)
子基板に74HC244を置く前提(08-24(5)C)なので相手の駆動力に依存しない。
ノイズ耐性とLレベルの確実性を優先。結線・部品・フットプリントは不変。

Co-Authored-By: Claude Opus 5 <noreply@anthropic.com>
Claude-Session: https://claude.ai/code/session_013dwHJLw3RmXmt8a4h9mnqw
Parts:
- RN1009, RN1010: value 47K -> 10K
Changed lines of the file:
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@@
 			)
 		)
-		(property "Value" "47K"
+		(property "Value" "10K"
 			(at 87.63 53.594 0)
 			(show_name no)
@@
 			)
 		)
-		(property "Value" "47K"
+		(property "Value" "10K"
 			(at 81.788 53.086 0)
 			(show_name no)
@@
 			)
 		)
-		(property "Value" "47K"
+		(property "Value" "10K"
 			(at 197.866 218.44 0)
 			(show_name no)
@@
 			)
 		)
-		(property "Value" "47K"
+		(property "Value" "10K"
 			(at 100.33 61.214 0)
 			(show_name no)
@@
 			)
 		)
-		(property "Value" "47K"
+		(property "Value" "10K"
 			(at 318.77 66.04 0)
 			(show_name no)
@@
 			)
 		)
-		(property "Value" "47K"
+		(property "Value" "10K"
 			(at 311.15 66.294 0)
 			(show_name no)
@@
 			)
 		)
-		(property "Value" "47K"
+		(property "Value" "10K"
 			(at 194.818 58.928 0)
 			(show_name no)
@@
 			)
 		)
-		(property "Value" "47K"
+		(property "Value" "10K"
 			(at 192.024 225.806 0)
 			(show_name no)
@@
 			)
 		)
-		(property "Value" "47K"
+		(property "Value" "10K"
 			(at 93.472 60.706 0)
 			(show_name no)
@@
 			)
 		)
-		(property "Value" "47K"
+		(property "Value" "10K"
 			(at 201.676 58.166 0)
 			(show_name no)
@@
 			)
 		)
-		(property "Value" "47K"
+		(property "Value" "10K"
 			(at 202.438 226.06 0)
 			(show_name no)
@@
 			)
 		)
-		(property "Value" "47K"
+		(property "Value" "10K"
 			(at 214.122 58.674 0)
 			(show_name no)
@@
 			)
 		)
-		(property "Value" "47K"
+		(property "Value" "10K"
 			(at 303.784 60.198 0)
 			(show_name no)
@@
 			)
 		)
-		(property "Value" "47K"
+		(property "Value" "10K"
 			(at 207.772 58.42 0)
 			(show_name no)
@@
 			)
 		)
-		(property "Value" "47K"
+		(property "Value" "10K"
 			(at 326.39 64.7699 0)
 			(show_name no)
@@
 			)
 		)
-		(property "Value" "47K"
+		(property "Value" "10K"
 			(at 209.296 225.552 0)
 			(show_name no)

Commit message: ver2: IF板のDIP直列1KΩ×16を削除／LED抵抗を8素子SIPへ集約(130→110部品)
SW1001-1004のpin5-8をVDD直結に戻し、R1001-1016を削除。
inPort/outPortのLED抵抗をR_Network04×4→R_Network08_Split×2へ集約。
検証は全項目合格(署名変化28件・未接続入力0・残骸ネット0・ERC 0/0)。

Co-Authored-By: Claude Opus 5 <noreply@anthropic.com>
Claude-Session: https://claude.ai/code/session_013dwHJLw3RmXmt8a4h9mnqw
Parts:
- removed R1001, R1002, R1003, R1004, R1005, R1006, R1007, R1008, R1009, R1010, R1011, R1012, R1013, R1014, R1015, R1016: 1K, Resistor_THT:R_Axial_DIN0207_L6.3mm_D2.5mm_P10.16mm_Horizontal, symbol Device:R
- removed RN1002, RN1003, RN1005, RN1007: 4.7K, Resistor_THT:R_Array_SIP5, symbol Device:R_Network04
- added RN1001, RN1002: 4.7K, Resistor_THT:R_Array_SIP9, symbol Device:R_Network08_Split
Connections:
- net GND: now also RN1001.1 (R1), RN1001.1 (R1), RN1001.1 (R1), RN1001.1 (R1), RN1001.1 (R1), RN1001.1 (R1), RN1001.1 (R1), RN1001.1 (R1), RN1002.1 (R1), RN1002.1 (R1), RN1002.1 (R1), RN1002.1 (R1), RN1002.1 (R1), RN1002.1 (R1), RN1002.1 (R1), RN1002.1 (R1)
- net VDD: now also SW1001.5, SW1001.6, SW1001.7, SW1001.8, SW1002.5, SW1002.6, SW1002.7, SW1002.8, SW1003.5, SW1003.6, SW1003.7, SW1003.8, SW1004.5, SW1004.6, SW1004.7, SW1004.8
- net at D1007.1 (K): now also RN1001.8 (R7.2)
- net at D1016.1 (K): now also RN1002.9 (R8.2)
- net at D1015.1 (K): now also RN1002.8 (R7.2)
- net at D1014.1 (K): now also RN1002.7 (R6.2)
- net at D1013.1 (K): now also RN1002.6 (R5.2)
- net at D1008.1 (K): now also RN1001.9 (R8.2)
- net at D1003.1 (K): now also RN1001.3 (R2.2)
- net at D1011.1 (K): now also RN1002.4 (R3.2)
- net at D1006.1 (K): now also RN1001.7 (R6.2)
- net at D1005.1 (K): now also RN1001.6 (R5.2)
- net at D1009.1 (K): now also RN1002.2 (R1.2)
- net at D1012.1 (K): now also RN1002.5 (R4.2)
- net at D1004.1 (K): now also RN1001.5 (R4.2)
- net at D1010.1 (K): now also RN1002.3 (R2.2)
- net at D1002.1 (K): now also RN1001.4 (R3.2)
- net at D1001.1 (K): now also RN1001.2 (R1.2)
