File: ver2/hardware/基板分割_0827/TB04addr8bit_if/outPut.kicad_sch (KiCad schematic)
At the start: 32 parts, among them J901 Conn_02x05_Odd_Even, J902 Conn_02x05_Odd_Even, J903 Conn_02x05_Odd_Even, J904 Conn_02x05_Odd_Even, U901 74LS377, U902 74LS377, U903 74LS377, U905 74LS377

Commit message: ver2: 3分割の74LS表記をHCへ一括変更(31パッケージ・Valueのみ)
- 書き換えたのはValueプロパティのみ(56件=31パッケージ)
- lib_id(74xx:74LS***)とDatasheetは変更せず。HC品のシンボルがKiCADに
  無いため、lib_idを変えるとシンボル未検出になる
- 74LS->74HCの単純置換で9品種すべて実在の型番(00/08/10/32/139/157/
  253/273/377)。ピン配置は同一でネットリストへの影響なし

検証: 残存する74LSのValue 0件、git diffの変更行はValueの56行のみ
申し送り: PCB側のValueは未同期。「回路図からPCBを更新」で解消する

Co-Authored-By: Claude Opus 5 <noreply@anthropic.com>
Parts:
- U901, U902, U903, U905: value 74LS377 -> 74HC377
Changed lines of the file:
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@@
 			)
 		)
-		(property "Value" "74LS377"
+		(property "Value" "74HC377"
 			(at 245.9833 167.64 0)
 			(show_name no)
@@
 			)
 		)
-		(property "Value" "74LS377"
+		(property "Value" "74HC377"
 			(at 242.1733 50.8 0)
 			(show_name no)
@@
 			)
 		)
-		(property "Value" "74LS377"
+		(property "Value" "74HC377"
 			(at 79.6133 52.07 0)
 			(show_name no)
@@
 			)
 		)
-		(property "Value" "74LS377"
+		(property "Value" "74HC377"
 			(at 83.4233 168.91 0)
 			(show_name no)

Commit message: ver2: IF板のDIP直列1KΩ×16を削除／LED抵抗を8素子SIPへ集約(130→110部品)
SW1001-1004のpin5-8をVDD直結に戻し、R1001-1016を削除。
inPort/outPortのLED抵抗をR_Network04×4→R_Network08_Split×2へ集約。
検証は全項目合格(署名変化28件・未接続入力0・残骸ネット0・ERC 0/0)。

Co-Authored-By: Claude Opus 5 <noreply@anthropic.com>
Claude-Session: https://claude.ai/code/session_013dwHJLw3RmXmt8a4h9mnqw
Parts:
- removed RN901, RN902, RN903, RN904: 4.7K, Resistor_THT:R_Array_SIP5, symbol Device:R_Network04
- added RN901, RN902: 4.7K, Resistor_THT:R_Array_SIP9, symbol Device:R_Network08_Split
Connections:
- net GND: now also RN901.1 (R1), RN901.1 (R1), RN901.1 (R1), RN901.1 (R1), RN901.1 (R1), RN901.1 (R1), RN901.1 (R1), RN901.1 (R1), RN902.1 (R1), RN902.1 (R1), RN902.1 (R1), RN902.1 (R1), RN902.1 (R1), RN902.1 (R1), RN902.1 (R1), RN902.1 (R1)
- net at D905.1 (K): now also RN901.6 (R5.2)
- net at D914.1 (K): now also RN902.7 (R6.2)
- net at D907.1 (K): now also RN901.8 (R7.2)
- net at D901.1 (K): now also RN901.2 (R1.2)
- net at D911.1 (K): now also RN902.4 (R3.2)
- net at D906.1 (K): now also RN901.7 (R6.2)
- net at D912.1 (K): now also RN902.5 (R4.2)
- net at D916.1 (K): now also RN902.9 (R8.2)
- net at D904.1 (K): now also RN901.5 (R4.2)
- net at D903.1 (K): now also RN901.3 (R2.2)
- net at D915.1 (K): now also RN902.8 (R7.2)
- net at D909.1 (K): now also RN902.2 (R1.2)
- net at D908.1 (K): now also RN901.9 (R8.2)
- net at D913.1 (K): now also RN902.6 (R5.2)
- net at D910.1 (K): now also RN902.3 (R2.2)
- net at D902.1 (K): now also RN901.4 (R3.2)
